Commit message: Fixed meshes and updated urdf

File: urdf/hdt_7dof_right.xacro (robot description, xacro)
@@ -16,5 +16,5 @@
 	<xacro:include filename="$(find hdt_7dof_description)/urdf/hdt_7dof.gazebo" /> -->
 	<!-- segment 0 -->
-	<link name="world"/>
+	<link name="base_link"/>
 	<!-- segment 1 -->
 	<joint name="joint1" type="revolute">
@@ -23,5 +23,5 @@
 		<limit effort="60.0" lower="-3.1416" upper="1.0472" velocity="2.0944"/>
 		<origin xyz="0 0 0" rpy="0 0 0"/>
-		<parent link="world"/>
+		<parent link="base_link"/>
 		<child link="link1"/>
     		<dynamics damping="0.7" friction="0.0"/>
