Commit message: Add gripper frames
The palm frame is very near the wrist. This new frame is near
the fingers, which makes planning easier.

File: urdf/hdt_7dof_left_macro.xacro (robot description, xacro)
@@ -459,4 +459,11 @@
 			<material>Gazebo/Black</material>
 		</gazebo>
+		<!-- gripper frame -->
+		<joint name="${prefix}gripper_frame_joint" type="fixed">
+			<origin xyz="0 -0.13 0" rpy="0 0 -1.57079" />
+			<parent link="${prefix}palm" />
+			<child link="${prefix}gripper_frame" />
+		</joint>
+		<link name="${prefix}gripper_frame" />
 		<!-- thumb base -->
 		<joint name="${prefix}thumb_base" type="revolute">

File: urdf/hdt_7dof_right_macro.xacro (robot description, xacro)
@@ -459,4 +459,11 @@
 			<material>Gazebo/Black</material>
 		</gazebo>
+		<!-- gripper frame -->
+		<joint name="${prefix}gripper_frame_joint" type="fixed">
+			<origin xyz="0 -0.13 0" rpy="0 0 -1.57079" />
+			<parent link="${prefix}palm" />
+			<child link="${prefix}gripper_frame" />
+		</joint>
+		<link name="${prefix}gripper_frame" />
 		<!-- thumb base -->
 		<joint name="${prefix}thumb_base" type="revolute">

Commit message: Fix some whitespace in macro files

File: urdf/hdt_7dof_left_macro.xacro (robot description, xacro)
@@ -4,7 +4,7 @@
 	<xacro:macro name="default_inertia">
 		<inertia
-		ixx="0.0005" ixy="0.0" ixz="0.0"
-		iyy="0.0005" iyz="0.0"
-		izz="0.0005"/>
+			ixx="0.0005" ixy="0.0" ixz="0.0"
+			iyy="0.0005" iyz="0.0"
+			izz="0.0005"/>
 	</xacro:macro>
 	<xacro:macro name="hdt_7dof_left" params="parent x y z yaw prefix">
@@ -53,10 +53,10 @@
 			</visual>
 			<inertial>
-			<origin xyz="-0.04488 0 0" rpy="0 0 0"/>
-			<mass value="1.00775"/>
-				<inertia
-				ixx="0.00064952" ixy="0.0" ixz="0.0"
-				iyy="0.00104342" iyz="0.0"
-				izz="0.00104342"/>
+				<origin xyz="-0.04488 0 0" rpy="0 0 0"/>
+				<mass value="1.00775"/>
+				<inertia
+					ixx="0.00064952" ixy="0.0" ixz="0.0"
+					iyy="0.00104342" iyz="0.0"
+					izz="0.00104342"/>
 			</inertial>
 		</link>
@@ -87,7 +87,7 @@
 				<mass value="0.66774822"/>
 				<inertia
-				ixx="0.00062987" ixy="0.0" ixz="0.0"
-				iyy="0.00091291" iyz="0.0"
-				izz="0.00110241"/>
+					ixx="0.00062987" ixy="0.0" ixz="0.0"
+					iyy="0.00091291" iyz="0.0"
+					izz="0.00110241"/>
 			</inertial>
 		</link>
@@ -132,7 +132,7 @@
 				<mass value="0.69896"/>
 				<inertia
-				ixx="0.00088116" ixy="0.0" ixz="0.0"
-				iyy="0.00094182" iyz="0.0"
-				izz="0.00032992"/>
+					ixx="0.00088116" ixy="0.0" ixz="0.0"
+					iyy="0.00094182" iyz="0.0"
+					izz="0.00032992"/>
 			</inertial>
 		</link>
@@ -177,7 +177,7 @@
 				<mass value="1.77733729"/>
 				<inertia
-				ixx="0.00450640" ixy="0.0" ixz="0.0"
-				iyy="0.00450640" iyz="0.0"
-				izz="0.00114447"/>
+					ixx="0.00450640" ixy="0.0" ixz="0.0"
+					iyy="0.00450640" iyz="0.0"
+					izz="0.00114447"/>
 			</inertial>
 		</link>
@@ -208,7 +208,7 @@
 				<mass value="0.66774822"/>
 				<inertia
-				ixx="0.00091291" ixy="0.0" ixz="0.0"
-				iyy="0.00110241" iyz="0.0"
-				izz="0.00062987"/>
+					ixx="0.00091291" ixy="0.0" ixz="0.0"
+					iyy="0.00110241" iyz="0.0"
+					izz="0.00062987"/>
 			</inertial>
 		</link>
@@ -253,7 +253,7 @@
 				<mass value="0.69896279"/>
 				<inertia
-				ixx="0.00094182" ixy="0.0" ixz="0.0"
-				iyy="0.00032992" iyz="0.0"
-				izz="0.00088116"/>
+					ixx="0.00094182" ixy="0.0" ixz="0.0"
+					iyy="0.00032992" iyz="0.0"
+					izz="0.00088116"/>
 			</inertial>
 		</link>
@@ -298,7 +298,7 @@
 				<mass value="1.00775488"/>
 				<inertia
-				ixx="0.00104342" ixy="0.0" ixz="0.0"
-				iyy="0.00064952" iyz="0.0"
-				izz="0.00104342"/>
+					ixx="0.00104342" ixy="0.0" ixz="0.0"
+					iyy="0.00064952" iyz="0.0"
+					izz="0.00104342"/>
 			</inertial>
 		</link>
@@ -329,7 +329,7 @@
 				<mass value="0.50058"/>
 				<inertia
-				ixx="0.000580228" ixy="0.0" ixz="0.0"
-				iyy="0.000541503" iyz="0.0"
-				izz="0.000750977"/>
+					ixx="0.000580228" ixy="0.0" ixz="0.0"
+					iyy="0.000541503" iyz="0.0"
+					izz="0.000750977"/>
 			</inertial>
 		</link>
@@ -374,7 +374,7 @@
 				<mass value="0.99934"/>
 				<inertia
-				ixx="0.001905243" ixy="0.0" ixz="0.0"
-				iyy="0.000474765" iyz="0.0"
-				izz="0.001905243"/>
+					ixx="0.001905243" ixy="0.0" ixz="0.0"
+					iyy="0.000474765" iyz="0.0"
+					izz="0.001905243"/>
 			</inertial>
 		</link>
@@ -419,7 +419,7 @@
 				<mass value="0.47608"/>
 				<inertia
-				ixx="0.000705091" ixy="0.0" ixz="0.0"
-				iyy="0.000537081" iyz="0.0"
-				izz="0.000534342"/>
+					ixx="0.000705091" ixy="0.0" ixz="0.0"
+					iyy="0.000537081" iyz="0.0"
+					izz="0.000534342"/>
 			</inertial>
 		</link>
@@ -451,7 +451,7 @@
 				<mass value="0.56756"/>
 				<inertia
-				ixx="0.001727803" ixy="0.000001205" ixz="0.0"
-				iyy="0.000549457" iyz="-0.000101997"
-				izz="0.001418031"/>
+					ixx="0.001727803" ixy="0.000001205" ixz="0.0"
+					iyy="0.000549457" iyz="-0.000101997"
+					izz="0.001418031"/>
 			</inertial>
 		</link>
@@ -503,7 +503,7 @@
 				<mass value="0.08562"/>
 				<inertia
-				ixx="0.0000315" ixy="0.0" ixz="0.0"
-				iyy="0.000034299" iyz="0.0"
-				izz="0.000022344"/>
+					ixx="0.0000315" ixy="0.0" ixz="0.0"
+					iyy="0.000034299" iyz="0.0"
+					izz="0.000022344"/>
 			</inertial>
 		</link>
@@ -549,7 +549,7 @@
 				<xacro:default_inertia />
 				<!-- <inertia
-				ixx="0.000004718" ixy="0.0" ixz="0.0"
-				iyy="0.000005374" iyz="-0.000000071"
-				izz="0.000002921"/> -->
+					ixx="0.000004718" ixy="0.0" ixz="0.0"
+					iyy="0.000005374" iyz="-0.000000071"
+					izz="0.000002921"/> -->
 			</inertial>
 		</link>
@@ -581,7 +581,7 @@
 				<mass value="0.0085"/>
 				<inertia
-				ixx="0.000001099" ixy="0.0" ixz="0.0"
-				iyy="0.000001639" iyz="0.000000096"
-				izz="0.000000981"/>
+					ixx="0.000001099" ixy="0.0" ixz="0.0"
+					iyy="0.000001639" iyz="0.000000096"
+					izz="0.000000981"/>
 			</inertial>
 		</link>
@@ -613,7 +613,7 @@
 				<mass value="0.0092"/>
 				<inertia
-				ixx="0.00000066" ixy="0.0" ixz="0.0"
-				iyy="0.000000837" iyz="0.0"
-				izz="0.000000695"/>
+					ixx="0.00000066" ixy="0.0" ixz="0.0"
+					iyy="0.000000837" iyz="0.0"
+					izz="0.000000695"/>
 			</inertial>
 		</link>
@@ -659,7 +659,7 @@
 				<xacro:default_inertia />
 				<!-- <inertia
-				ixx="0.000005374" ixy="-0.000000071" ixz="0.0"
-				iyy="0.000002921" iyz="0.0"
-				izz="0.000004718"/> -->
+					ixx="0.000005374" ixy="-0.000000071" ixz="0.0"
+					iyy="0.000002921" iyz="0.0"
+					izz="0.000004718"/> -->
 			</inertial>
 		</link>
@@ -691,7 +691,7 @@
 				<mass value="0.0085"/>
 				<inertia
-				ixx="0.000001639" ixy="0.000000096" ixz="0.0"
-				iyy="0.000000981" iyz="0.0"
-				izz="0.000001099"/>
+					ixx="0.000001639" ixy="0.000000096" ixz="0.0"
+					iyy="0.000000981" iyz="0.0"
+					izz="0.000001099"/>
 			</inertial>
 		</link>
@@ -723,7 +723,7 @@
 				<mass value="0.0092"/>
 				<inertia
-				ixx="0.000000837" ixy="0.0" ixz="0.0"
-				iyy="0.000000695" iyz="0.0"
-				izz="0.00000066"/>
+					ixx="0.000000837" ixy="0.0" ixz="0.0"
+					iyy="0.000000695" iyz="0.0"
+					izz="0.00000066"/>
 			</inertial>
 		</link>
@@ -769,7 +769,7 @@
 				<xacro:default_inertia />
 				<!-- <inertia
-				ixx="0.000005374" ixy="-0.000000071" ixz="0.0"
-				iyy="0.000002921" iyz="0.0"
-				izz="0.000004718"/> -->
+					ixx="0.000005374" ixy="-0.000000071" ixz="0.0"
+					iyy="0.000002921" iyz="0.0"
+					izz="0.000004718"/> -->
 			</inertial>
 		</link>
@@ -801,7 +801,7 @@
 				<mass value="0.0085"/>
 				<inertia
-				ixx="0.000001639" ixy="0.000000096" ixz="0.0"
-				iyy="0.000000981" iyz="0.0"
-				izz="0.000001099"/>
+					ixx="0.000001639" ixy="0.000000096" ixz="0.0"
+					iyy="0.000000981" iyz="0.0"
+					izz="0.000001099"/>
 			</inertial>
 		</link>
@@ -833,7 +833,7 @@
 				<mass value="0.0092"/>
 				<inertia
-				ixx="0.000000837" ixy="0.0" ixz="0.0"
-				iyy="0.000000695" iyz="0.0"
-				izz="0.00000066"/>
+					ixx="0.000000837" ixy="0.0" ixz="0.0"
+					iyy="0.000000695" iyz="0.0"
+					izz="0.00000066"/>
 			</inertial>
 		</link>

File: urdf/hdt_7dof_right_macro.xacro (robot description, xacro)
@@ -4,7 +4,7 @@
 	<xacro:macro name="default_inertia">
 		<inertia
-		ixx="0.0005" ixy="0.0" ixz="0.0"
-		iyy="0.0005" iyz="0.0"
-		izz="0.0005"/>
+			ixx="0.0005" ixy="0.0" ixz="0.0"
+			iyy="0.0005" iyz="0.0"
+			izz="0.0005"/>
 	</xacro:macro>
 	<xacro:macro name="hdt_7dof_right" params="parent x y z yaw prefix">
@@ -53,10 +53,10 @@
 			</visual>
 			<inertial>
-			<origin xyz="-0.04488 0 0" rpy="0 0 0"/>
-			<mass value="1.00775"/>
-				<inertia
-				ixx="0.00064952" ixy="0.0" ixz="0.0"
-				iyy="0.00104342" iyz="0.0"
-				izz="0.00104342"/>
+				<origin xyz="-0.04488 0 0" rpy="0 0 0"/>
+				<mass value="1.00775"/>
+				<inertia
+					ixx="0.00064952" ixy="0.0" ixz="0.0"
+					iyy="0.00104342" iyz="0.0"
+					izz="0.00104342"/>
 			</inertial>
 		</link>
@@ -87,7 +87,7 @@
 				<mass value="0.66774822"/>
 				<inertia
-				ixx="0.00062987" ixy="0.0" ixz="0.0"
-				iyy="0.00091291" iyz="0.0"
-				izz="0.00110241"/>
+					ixx="0.00062987" ixy="0.0" ixz="0.0"
+					iyy="0.00091291" iyz="0.0"
+					izz="0.00110241"/>
 			</inertial>
 		</link>
@@ -132,7 +132,7 @@
 				<mass value="0.69896"/>
 				<inertia
-				ixx="0.00088116" ixy="0.0" ixz="0.0"
-				iyy="0.00094182" iyz="0.0"
-				izz="0.00032992"/>
+					ixx="0.00088116" ixy="0.0" ixz="0.0"
+					iyy="0.00094182" iyz="0.0"
+					izz="0.00032992"/>
 			</inertial>
 		</link>
@@ -177,7 +177,7 @@
 				<mass value="1.77733729"/>
 				<inertia
-				ixx="0.00450640" ixy="0.0" ixz="0.0"
-				iyy="0.00450640" iyz="0.0"
-				izz="0.00114447"/>
+					ixx="0.00450640" ixy="0.0" ixz="0.0"
+					iyy="0.00450640" iyz="0.0"
+					izz="0.00114447"/>
 			</inertial>
 		</link>
@@ -208,7 +208,7 @@
 				<mass value="0.66774822"/>
 				<inertia
-				ixx="0.00091291" ixy="0.0" ixz="0.0"
-				iyy="0.00110241" iyz="0.0"
-				izz="0.00062987"/>
+					ixx="0.00091291" ixy="0.0" ixz="0.0"
+					iyy="0.00110241" iyz="0.0"
+					izz="0.00062987"/>
 			</inertial>
 		</link>
@@ -253,7 +253,7 @@
 				<mass value="0.69896279"/>
 				<inertia
-				ixx="0.00094182" ixy="0.0" ixz="0.0"
-				iyy="0.00032992" iyz="0.0"
-				izz="0.00088116"/>
+					ixx="0.00094182" ixy="0.0" ixz="0.0"
+					iyy="0.00032992" iyz="0.0"
+					izz="0.00088116"/>
 			</inertial>
 		</link>
@@ -298,7 +298,7 @@
 				<mass value="1.00775488"/>
 				<inertia
-				ixx="0.00104342" ixy="0.0" ixz="0.0"
-				iyy="0.00064952" iyz="0.0"
-				izz="0.00104342"/>
+					ixx="0.00104342" ixy="0.0" ixz="0.0"
+					iyy="0.00064952" iyz="0.0"
+					izz="0.00104342"/>
 			</inertial>
 		</link>
@@ -329,7 +329,7 @@
 				<mass value="0.50058"/>
 				<inertia
-				ixx="0.000580228" ixy="0.0" ixz="0.0"
-				iyy="0.000541503" iyz="0.0"
-				izz="0.000750977"/>
+					ixx="0.000580228" ixy="0.0" ixz="0.0"
+					iyy="0.000541503" iyz="0.0"
+					izz="0.000750977"/>
 			</inertial>
 		</link>
@@ -374,7 +374,7 @@
 				<mass value="0.99934"/>
 				<inertia
-				ixx="0.001905243" ixy="0.0" ixz="0.0"
-				iyy="0.000474765" iyz="0.0"
-				izz="0.001905243"/>
+					ixx="0.001905243" ixy="0.0" ixz="0.0"
+					iyy="0.000474765" iyz="0.0"
+					izz="0.001905243"/>
 			</inertial>
 		</link>
@@ -419,7 +419,7 @@
 				<mass value="0.47608"/>
 				<inertia
-				ixx="0.000705091" ixy="0.0" ixz="0.0"
-				iyy="0.000537081" iyz="0.0"
-				izz="0.000534342"/>
+					ixx="0.000705091" ixy="0.0" ixz="0.0"
+					iyy="0.000537081" iyz="0.0"
+					izz="0.000534342"/>
 			</inertial>
 		</link>
@@ -451,7 +451,7 @@
 				<mass value="0.56756"/>
 				<inertia
-				ixx="0.001727803" ixy="0.000001205" ixz="0.0"
-				iyy="0.000549457" iyz="-0.000101997"
-				izz="0.001418031"/>
+					ixx="0.001727803" ixy="0.000001205" ixz="0.0"
+					iyy="0.000549457" iyz="-0.000101997"
+					izz="0.001418031"/>
 			</inertial>
 		</link>
@@ -503,7 +503,7 @@
 				<mass value="0.08562"/>
 				<inertia
-				ixx="0.0000315" ixy="0.0" ixz="0.0"
-				iyy="0.000034299" iyz="0.0"
-				izz="0.000022344"/>
+					ixx="0.0000315" ixy="0.0" ixz="0.0"
+					iyy="0.000034299" iyz="0.0"
+					izz="0.000022344"/>
 			</inertial>
 		</link>
@@ -549,7 +549,7 @@
 				<xacro:default_inertia />
 				<!-- <inertia
-				ixx="0.000004718" ixy="0.0" ixz="0.0"
-				iyy="0.000005374" iyz="-0.000000071"
-				izz="0.000002921"/> -->
+					ixx="0.000004718" ixy="0.0" ixz="0.0"
+					iyy="0.000005374" iyz="-0.000000071"
+					izz="0.000002921"/> -->
 			</inertial>
 		</link>
@@ -581,7 +581,7 @@
 				<mass value="0.0085"/>
 				<inertia
-				ixx="0.000001099" ixy="0.0" ixz="0.0"
-				iyy="0.000001639" iyz="0.000000096"
-				izz="0.000000981"/>
+					ixx="0.000001099" ixy="0.0" ixz="0.0"
+					iyy="0.000001639" iyz="0.000000096"
+					izz="0.000000981"/>
 			</inertial>
 		</link>
@@ -613,7 +613,7 @@
 				<mass value="0.0092"/>
 				<inertia
-				ixx="0.00000066" ixy="0.0" ixz="0.0"
-				iyy="0.000000837" iyz="0.0"
-				izz="0.000000695"/>
+					ixx="0.00000066" ixy="0.0" ixz="0.0"
+					iyy="0.000000837" iyz="0.0"
+					izz="0.000000695"/>
 			</inertial>
 		</link>
@@ -659,7 +659,7 @@
 				<xacro:default_inertia />
 				<!-- <inertia
-				ixx="0.000005374" ixy="-0.000000071" ixz="0.0"
-				iyy="0.000002921" iyz="0.0"
-				izz="0.000004718"/> -->
+					ixx="0.000005374" ixy="-0.000000071" ixz="0.0"
+					iyy="0.000002921" iyz="0.0"
+					izz="0.000004718"/> -->
 			</inertial>
 		</link>
@@ -691,7 +691,7 @@
 				<mass value="0.0085"/>
 				<inertia
-				ixx="0.000001639" ixy="0.000000096" ixz="0.0"
-				iyy="0.000000981" iyz="0.0"
-				izz="0.000001099"/>
+					ixx="0.000001639" ixy="0.000000096" ixz="0.0"
+					iyy="0.000000981" iyz="0.0"
+					izz="0.000001099"/>
 			</inertial>
 		</link>
@@ -723,7 +723,7 @@
 				<mass value="0.0092"/>
 				<inertia
-				ixx="0.000000837" ixy="0.0" ixz="0.0"
-				iyy="0.000000695" iyz="0.0"
-				izz="0.00000066"/>
+					ixx="0.000000837" ixy="0.0" ixz="0.0"
+					iyy="0.000000695" iyz="0.0"
+					izz="0.00000066"/>
 			</inertial>
 		</link>
@@ -769,7 +769,7 @@
 				<xacro:default_inertia />
 				<!-- <inertia
-				ixx="0.000005374" ixy="-0.000000071" ixz="0.0"
-				iyy="0.000002921" iyz="0.0"
-				izz="0.000004718"/> -->
+					ixx="0.000005374" ixy="-0.000000071" ixz="0.0"
+					iyy="0.000002921" iyz="0.0"
+					izz="0.000004718"/> -->
 			</inertial>
 		</link>
@@ -801,7 +801,7 @@
 				<mass value="0.0085"/>
 				<inertia
-				ixx="0.000001639" ixy="0.000000096" ixz="0.0"
-				iyy="0.000000981" iyz="0.0"
-				izz="0.000001099"/>
+					ixx="0.000001639" ixy="0.000000096" ixz="0.0"
+					iyy="0.000000981" iyz="0.0"
+					izz="0.000001099"/>
 			</inertial>
 		</link>
@@ -833,7 +833,7 @@
 				<mass value="0.0092"/>
 				<inertia
-				ixx="0.000000837" ixy="0.0" ixz="0.0"
-				iyy="0.000000695" iyz="0.0"
-				izz="0.00000066"/>
+					ixx="0.000000837" ixy="0.0" ixz="0.0"
+					iyy="0.000000695" iyz="0.0"
+					izz="0.00000066"/>
 			</inertial>
 		</link>
