Commit message: Make joint names more descriptive

File: urdf/hdt_7dof_left_macro.xacro (robot description, xacro)
@@ -19,6 +19,6 @@
 			<color rgba="${40/255} ${40/255} ${40/255} 1.0"/>
 		</material>
-		<!-- segment 1 -->
-		<joint name="${prefix}joint1" type="revolute">
+		<!-- shoulder -->
+		<joint name="${prefix}shoulder_pitch" type="revolute">
 			<hdt id="41" kmin="100" kmax="200" inertia="0.1"/>
 			<axis xyz="-1 0 0"/>
@@ -31,5 +31,5 @@
 		<transmission name="${prefix}tran1">
 			<type>transmission_interface/SimpleTransmission</type>
-			<joint name="${prefix}joint1">
+			<joint name="${prefix}shoulder_pitch">
 				<hardwareInterface>EffortJointInterface</hardwareInterface>
 			</joint>
@@ -95,6 +95,6 @@
 			<material>Gazebo/Black</material>
 		</gazebo>
-		<!-- segment 2 -->
-		<joint name="${prefix}joint2" type="revolute">
+		<!-- shoulder roll -->
+		<joint name="${prefix}shoulder_roll" type="revolute">
 			<hdt id="42" kmin="100" kmax="200" inertia="0.1"/>
 			<axis xyz="0 1 0"/>
@@ -107,5 +107,5 @@
 		<transmission name="${prefix}tran2">
 			<type>transmission_interface/SimpleTransmission</type>
-			<joint name="${prefix}joint2">
+			<joint name="${prefix}shoulder_roll">
 				<hardwareInterface>EffortJointInterface</hardwareInterface>
 			</joint>
@@ -140,6 +140,6 @@
 			<material>Gazebo/Grey</material>
 		</gazebo>
-		<!-- segment 3 -->
-		<joint name="${prefix}joint3" type="revolute">
+		<!-- upper arm -->
+		<joint name="${prefix}shoulder_yaw" type="revolute">
 			<hdt id="43" kmin="75" kmax="150" inertia="0.075"/>
 			<axis xyz="0 0 1"/>
@@ -152,5 +152,5 @@
 		<transmission name="${prefix}tran3">
 			<type>transmission_interface/SimpleTransmission</type>
-			<joint name="${prefix}joint3">
+			<joint name="${prefix}shoulder_yaw">
 				<hardwareInterface>EffortJointInterface</hardwareInterface>
 			</joint>
@@ -216,6 +216,6 @@
 			<material>Gazebo/Black</material>
 		</gazebo>
-		<!-- segment 4 -->
-		<joint name="${prefix}joint4" type="revolute">
+		<!-- elbow pitch -->
+		<joint name="${prefix}elbow_pitch" type="revolute">
 			<hdt id="44" kmin="75" kmax="150" inertia="0.075"/>
 			<axis xyz="-1 0 0"/>
@@ -228,5 +228,5 @@
 		<transmission name="${prefix}tran4">
 			<type>transmission_interface/SimpleTransmission</type>
-			<joint name="${prefix}joint4">
+			<joint name="${prefix}elbow_pitch">
 				<hardwareInterface>EffortJointInterface</hardwareInterface>
 			</joint>
@@ -261,6 +261,6 @@
 			<material>Gazebo/Grey</material>
 		</gazebo>
-		<!-- segment 5 -->
-		<joint name="${prefix}joint5" type="revolute">
+		<!-- forearm -->
+		<joint name="${prefix}elbow_roll" type="revolute">
 			<hdt id="45" kmin="50" kmax="100" inertia="0.05"/>
 			<axis xyz="0 -1 0"/>
@@ -273,5 +273,5 @@
 		<transmission name="${prefix}tran5">
 			<type>transmission_interface/SimpleTransmission</type>
-			<joint name="${prefix}joint5">
+			<joint name="${prefix}elbow_roll">
 				<hardwareInterface>EffortJointInterface</hardwareInterface>
 			</joint>
@@ -337,6 +337,6 @@
 			<material>Gazebo/Black</material>
 		</gazebo>
-		<!-- segment 6 -->
-		<joint name="${prefix}joint6" type="revolute">
+		<!-- wrist pitch -->
+		<joint name="${prefix}wrist_pitch" type="revolute">
 			<hdt id="46" kmin="50" kmax="100" inertia="0.05"/>
 			<axis xyz="1 0 0"/>
@@ -349,5 +349,5 @@
 		<transmission name="${prefix}tran6">
 			<type>transmission_interface/SimpleTransmission</type>
-			<joint name="${prefix}joint6">
+			<joint name="${prefix}wrist_pitch">
 				<hardwareInterface>EffortJointInterface</hardwareInterface>
 			</joint>
@@ -382,6 +382,6 @@
 			<material>Gazebo/Grey</material>
 		</gazebo>
-		<!-- segment 7 -->
-		<joint name="${prefix}joint7" type="revolute">
+		<!-- wrist yaw -->
+		<joint name="${prefix}wrist_yaw" type="revolute">
 			<hdt id="47" kmin="50" kmax="100" inertia="0.05"/>
 			<axis xyz="0 0 1"/>
@@ -394,5 +394,5 @@
 		<transmission name="${prefix}tran7">
 			<type>transmission_interface/SimpleTransmission</type>
-			<joint name="${prefix}joint7">
+			<joint name="${prefix}wrist_yaw">
 				<hardwareInterface>EffortJointInterface</hardwareInterface>
 			</joint>
@@ -467,5 +467,5 @@
 		<link name="${prefix}gripper_frame" />
 		<!-- thumb base -->
-		<joint name="${prefix}thumb_base" type="revolute">
+		<joint name="${prefix}thumb_roll" type="revolute">
 			<hdt id="50" kmin="5" kmax="20" inertia="0.01"/>
 			<axis xyz="0 -1 0"/>
@@ -478,5 +478,5 @@
 		<transmission name="${prefix}tran10">
 			<type>transmission_interface/SimpleTransmission</type>
-			<joint name="${prefix}thumb_base">
+			<joint name="${prefix}thumb_roll">
 				<hardwareInterface>EffortJointInterface</hardwareInterface>
 			</joint>
@@ -512,5 +512,5 @@
 		</gazebo>
 		<!-- thumb prox -->
-		<joint name="${prefix}thumb_prox" type="revolute">
+		<joint name="${prefix}thumb_pitch" type="revolute">
 			<hdt id="51" kmin="5" kmax="20" inertia="0.01"/>
 			<axis xyz="1 0 0"/>
@@ -523,5 +523,5 @@
 		<transmission name="${prefix}tran11">
 			<type>transmission_interface/SimpleTransmission</type>
-			<joint name="${prefix}thumb_prox">
+			<joint name="${prefix}thumb_pitch">
 				<hardwareInterface>EffortJointInterface</hardwareInterface>
 			</joint>
@@ -622,5 +622,5 @@
 		</gazebo>
 		<!-- index prox -->
-		<joint name="${prefix}index_prox" type="revolute">
+		<joint name="${prefix}index_yaw" type="revolute">
 			<hdt id="52" kmin="5" kmax="20" inertia="0.01"/>
 			<axis xyz="0 0 -1"/>
@@ -633,5 +633,5 @@
 		<transmission name="${prefix}tran12">
 			<type>transmission_interface/SimpleTransmission</type>
-			<joint name="${prefix}index_prox">
+			<joint name="${prefix}index_yaw">
 				<hardwareInterface>EffortJointInterface</hardwareInterface>
 			</joint>
@@ -732,5 +732,5 @@
 		</gazebo>
 		<!-- ring prox -->
-		<joint name="${prefix}ring_prox" type="revolute">
+		<joint name="${prefix}ring_yaw" type="revolute">
 			<hdt id="53" kmin="5" kmax="20" inertia="0.01"/>
 			<axis xyz="0 0 -1"/>
@@ -743,5 +743,5 @@
 		<transmission name="${prefix}tran13">
 			<type>transmission_interface/SimpleTransmission</type>
-			<joint name="${prefix}ring_prox">
+			<joint name="${prefix}ring_yaw">
 				<hardwareInterface>EffortJointInterface</hardwareInterface>
 			</joint>

File: urdf/hdt_7dof_right_macro.xacro (robot description, xacro)
@@ -19,6 +19,6 @@
 			<color rgba="${40/255} ${40/255} ${40/255} 1.0"/>
 		</material>
-		<!-- segment 1 -->
-		<joint name="${prefix}joint1" type="revolute">
+		<!-- shoulder -->
+		<joint name="${prefix}shoulder_pitch" type="revolute">
 			<hdt id="1" kmin="100" kmax="200" inertia="0.1"/>
 			<axis xyz="1 0 0"/>
@@ -31,5 +31,5 @@
 		<transmission name="${prefix}tran1">
 			<type>transmission_interface/SimpleTransmission</type>
-			<joint name="${prefix}joint1">
+			<joint name="${prefix}shoulder_pitch">
 				<hardwareInterface>EffortJointInterface</hardwareInterface>
 			</joint>
@@ -95,6 +95,6 @@
 			<material>Gazebo/Black</material>
 		</gazebo>
-		<!-- segment 2 -->
-		<joint name="${prefix}joint2" type="revolute">
+		<!-- shoulder roll -->
+		<joint name="${prefix}shoulder_roll" type="revolute">
 			<hdt id="2" kmin="100" kmax="200" inertia="0.1"/>
 			<axis xyz="0 -1 0"/>
@@ -107,5 +107,5 @@
 		<transmission name="${prefix}tran2">
 			<type>transmission_interface/SimpleTransmission</type>
-			<joint name="${prefix}joint2">
+			<joint name="${prefix}shoulder_roll">
 				<hardwareInterface>EffortJointInterface</hardwareInterface>
 			</joint>
@@ -140,6 +140,6 @@
 			<material>Gazebo/Grey</material>
 		</gazebo>
-		<!-- segment 3 -->
-		<joint name="${prefix}joint3" type="revolute">
+		<!-- upper arm -->
+		<joint name="${prefix}shoulder_yaw" type="revolute">
 			<hdt id="3" kmin="75" kmax="150" inertia="0.075"/>
 			<axis xyz="0 0 1"/>
@@ -152,5 +152,5 @@
 		<transmission name="${prefix}tran3">
 			<type>transmission_interface/SimpleTransmission</type>
-			<joint name="${prefix}joint3">
+			<joint name="${prefix}shoulder_yaw">
 				<hardwareInterface>EffortJointInterface</hardwareInterface>
 			</joint>
@@ -216,6 +216,6 @@
 			<material>Gazebo/Black</material>
 		</gazebo>
-		<!-- segment 4 -->
-		<joint name="${prefix}joint4" type="revolute">
+		<!-- elbow pitch -->
+		<joint name="${prefix}elbow_pitch" type="revolute">
 			<hdt id="4" kmin="75" kmax="150" inertia="0.075"/>
 			<axis xyz="1 0 0"/>
@@ -228,5 +228,5 @@
 		<transmission name="${prefix}tran4">
 			<type>transmission_interface/SimpleTransmission</type>
-			<joint name="${prefix}joint4">
+			<joint name="${prefix}elbow_pitch">
 				<hardwareInterface>EffortJointInterface</hardwareInterface>
 			</joint>
@@ -261,6 +261,6 @@
 			<material>Gazebo/Grey</material>
 		</gazebo>
-		<!-- segment 5 -->
-		<joint name="${prefix}joint5" type="revolute">
+		<!-- forearm -->
+		<joint name="${prefix}elbow_roll" type="revolute">
 			<hdt id="5" kmin="50" kmax="100" inertia="0.05"/>
 			<axis xyz="0 -1 0"/>
@@ -273,5 +273,5 @@
 		<transmission name="${prefix}tran5">
 			<type>transmission_interface/SimpleTransmission</type>
-			<joint name="${prefix}joint5">
+			<joint name="${prefix}elbow_roll">
 				<hardwareInterface>EffortJointInterface</hardwareInterface>
 			</joint>
@@ -337,6 +337,6 @@
 			<material>Gazebo/Black</material>
 		</gazebo>
-		<!-- segment 6 -->
-		<joint name="${prefix}joint6" type="revolute">
+		<!-- wrist pitch -->
+		<joint name="${prefix}wrist_pitch" type="revolute">
 			<hdt id="6" kmin="50" kmax="100" inertia="0.05"/>
 			<axis xyz="1 0 0"/>
@@ -349,5 +349,5 @@
 		<transmission name="${prefix}tran6">
 			<type>transmission_interface/SimpleTransmission</type>
-			<joint name="${prefix}joint6">
+			<joint name="${prefix}wrist_pitch">
 				<hardwareInterface>EffortJointInterface</hardwareInterface>
 			</joint>
@@ -382,6 +382,6 @@
 			<material>Gazebo/Grey</material>
 		</gazebo>
-		<!-- segment 7 -->
-		<joint name="${prefix}joint7" type="revolute">
+		<!-- wrist yaw -->
+		<joint name="${prefix}wrist_yaw" type="revolute">
 			<hdt id="7" kmin="50" kmax="100" inertia="0.05"/>
 			<axis xyz="0 0 1"/>
@@ -394,5 +394,5 @@
 		<transmission name="${prefix}tran7">
 			<type>transmission_interface/SimpleTransmission</type>
-			<joint name="${prefix}joint7">
+			<joint name="${prefix}wrist_yaw">
 				<hardwareInterface>EffortJointInterface</hardwareInterface>
 			</joint>
@@ -467,5 +467,5 @@
 		<link name="${prefix}gripper_frame" />
 		<!-- thumb base -->
-		<joint name="${prefix}thumb_base" type="revolute">
+		<joint name="${prefix}thumb_roll" type="revolute">
 			<hdt id="10" kmin="5" kmax="20" inertia="0.01"/>
 			<axis xyz="0 -1 0"/>
@@ -478,5 +478,5 @@
 		<transmission name="${prefix}tran10">
 			<type>transmission_interface/SimpleTransmission</type>
-			<joint name="${prefix}thumb_base">
+			<joint name="${prefix}thumb_roll">
 				<hardwareInterface>EffortJointInterface</hardwareInterface>
 			</joint>
@@ -512,5 +512,5 @@
 		</gazebo>
 		<!-- thumb prox -->
-		<joint name="${prefix}thumb_prox" type="revolute">
+		<joint name="${prefix}thumb_pitch" type="revolute">
 			<hdt id="11" kmin="5" kmax="20" inertia="0.01"/>
 			<axis xyz="1 0 0"/>
@@ -523,5 +523,5 @@
 		<transmission name="${prefix}tran11">
 			<type>transmission_interface/SimpleTransmission</type>
-			<joint name="${prefix}thumb_prox">
+			<joint name="${prefix}thumb_pitch">
 				<hardwareInterface>EffortJointInterface</hardwareInterface>
 			</joint>
@@ -622,5 +622,5 @@
 		</gazebo>
 		<!-- index prox -->
-		<joint name="${prefix}index_prox" type="revolute">
+		<joint name="${prefix}index_yaw" type="revolute">
 			<hdt id="12" kmin="5" kmax="20" inertia="0.01"/>
 			<axis xyz="0 0 1"/>
@@ -633,5 +633,5 @@
 		<transmission name="${prefix}tran12">
 			<type>transmission_interface/SimpleTransmission</type>
-			<joint name="${prefix}index_prox">
+			<joint name="${prefix}index_yaw">
 				<hardwareInterface>EffortJointInterface</hardwareInterface>
 			</joint>
@@ -732,5 +732,5 @@
 		</gazebo>
 		<!-- ring prox -->
-		<joint name="${prefix}ring_prox" type="revolute">
+		<joint name="${prefix}ring_yaw" type="revolute">
 			<hdt id="13" kmin="5" kmax="20" inertia="0.01"/>
 			<axis xyz="0 0 1"/>
@@ -743,5 +743,5 @@
 		<transmission name="${prefix}tran13">
 			<type>transmission_interface/SimpleTransmission</type>
-			<joint name="${prefix}ring_prox">
+			<joint name="${prefix}ring_yaw">
 				<hardwareInterface>EffortJointInterface</hardwareInterface>
 			</joint>

Commit message: Change default_inertia to default_inertial (the parent xml node)

File: urdf/hdt_7dof_left_macro.xacro (robot description, xacro)
@@ -2,9 +2,12 @@
 <robot name="hdt_7dof" xmlns:xacro="http://www.ros.org/wiki/xacro">
 	<!-- default inertia -->
-	<xacro:macro name="default_inertia">
-		<inertia
-			ixx="0.0005" ixy="0.0" ixz="0.0"
-			iyy="0.0005" iyz="0.0"
-			izz="0.0005"/>
+	<xacro:macro name="default_inertial">
+		<inertial>
+			<mass value="0.025"/>
+			<inertia
+				ixx="0.0005" ixy="0.0" ixz="0.0"
+				iyy="0.0005" iyz="0.0"
+				izz="0.0005"/>
+		</inertial>
 	</xacro:macro>
 	<xacro:macro name="hdt_7dof_left" params="parent x y z yaw prefix">
@@ -544,13 +547,5 @@
 				<material name="${prefix}grey"/>
 			</visual>
-			<inertial>
-				<origin xyz="0 0.001 0.02063" rpy="0 0 0"/>
-				<mass value="0.02523"/>
-				<xacro:default_inertia />
-				<!-- <inertia
-					ixx="0.000004718" ixy="0.0" ixz="0.0"
-					iyy="0.000005374" iyz="-0.000000071"
-					izz="0.000002921"/> -->
-			</inertial>
+			<xacro:default_inertial/>
 		</link>
 		<gazebo reference="${prefix}thumb_prox">
@@ -654,13 +649,5 @@
 				<material name="${prefix}grey"/>
 			</visual>
-			<inertial>
-				<origin xyz="-0.001 -0.02063 0" rpy="0 0 0"/>
-				<mass value="0.02523"/>
-				<xacro:default_inertia />
-				<!-- <inertia
-					ixx="0.000005374" ixy="-0.000000071" ixz="0.0"
-					iyy="0.000002921" iyz="0.0"
-					izz="0.000004718"/> -->
-			</inertial>
+			<xacro:default_inertial/>
 		</link>
 		<gazebo reference="${prefix}index_prox">
@@ -764,13 +751,5 @@
 				<material name="${prefix}grey"/>
 			</visual>
-			<inertial>
-				<origin xyz="-0.001 -0.02063 0" rpy="0 0 0"/>
-				<mass value="0.02523"/>
-				<xacro:default_inertia />
-				<!-- <inertia
-					ixx="0.000005374" ixy="-0.000000071" ixz="0.0"
-					iyy="0.000002921" iyz="0.0"
-					izz="0.000004718"/> -->
-			</inertial>
+			<xacro:default_inertial/>
 		</link>
 		<gazebo reference="${prefix}ring_prox">

File: urdf/hdt_7dof_right_macro.xacro (robot description, xacro)
@@ -2,9 +2,12 @@
 <robot name="hdt_7dof" xmlns:xacro="http://www.ros.org/wiki/xacro">
 	<!-- default inertia -->
-	<xacro:macro name="default_inertia">
-		<inertia
-			ixx="0.0005" ixy="0.0" ixz="0.0"
-			iyy="0.0005" iyz="0.0"
-			izz="0.0005"/>
+	<xacro:macro name="default_inertial">
+		<inertial>
+			<mass value="0.025"/>
+			<inertia
+				ixx="0.0005" ixy="0.0" ixz="0.0"
+				iyy="0.0005" iyz="0.0"
+				izz="0.0005"/>
+		</inertial>
 	</xacro:macro>
 	<xacro:macro name="hdt_7dof_right" params="parent x y z yaw prefix">
@@ -544,13 +547,5 @@
 				<material name="${prefix}grey"/>
 			</visual>
-			<inertial>
-				<origin xyz="0 0.001 0.02063" rpy="0 0 0"/>
-				<mass value="0.02523"/>
-				<xacro:default_inertia />
-				<!-- <inertia
-					ixx="0.000004718" ixy="0.0" ixz="0.0"
-					iyy="0.000005374" iyz="-0.000000071"
-					izz="0.000002921"/> -->
-			</inertial>
+			<xacro:default_inertial/>
 		</link>
 		<gazebo reference="${prefix}thumb_prox">
@@ -654,13 +649,5 @@
 				<material name="${prefix}grey"/>
 			</visual>
-			<inertial>
-				<origin xyz="-0.001 -0.02063 0" rpy="0 0 0"/>
-				<mass value="0.02523"/>
-				<xacro:default_inertia />
-				<!-- <inertia
-					ixx="0.000005374" ixy="-0.000000071" ixz="0.0"
-					iyy="0.000002921" iyz="0.0"
-					izz="0.000004718"/> -->
-			</inertial>
+			<xacro:default_inertial/>
 		</link>
 		<gazebo reference="${prefix}index_prox">
@@ -764,13 +751,5 @@
 				<material name="${prefix}grey"/>
 			</visual>
-			<inertial>
-				<origin xyz="-0.001 -0.02063 0" rpy="0 0 0"/>
-				<mass value="0.02523"/>
-				<xacro:default_inertia />
-				<!-- <inertia
-					ixx="0.000005374" ixy="-0.000000071" ixz="0.0"
-					iyy="0.000002921" iyz="0.0"
-					izz="0.000004718"/> -->
-			</inertial>
+			<xacro:default_inertial/>
 		</link>
 		<gazebo reference="${prefix}ring_prox">
