Commit message: Hacking in a ViGIR specific gripper frame.

File: urdf/hdt_7dof_hand.xacro (robot description, xacro)
@@ -45,4 +45,11 @@
         </joint>
         <link name="${prefix}gripper_frame" />
+        <!-- Hacked in joint to match ViGIR frames -->
+        <joint name="${prefix}vigir_joint" type="fixed">
+            <origin xyz = "0 -0.13 0" rpy="0 0 0" />
+            <parent link="${prefix}palm" />
+            <child link="${prefix}vigir_gripper" />
+        </joint>
+        <link name="${prefix}vigir_gripper" />
         <!-- thumb base -->
         <joint name="${prefix}thumb_roll" type="revolute">

Commit message: Renaming ViGIR links internally.

File: urdf/hdt_7dof_hand.xacro (robot description, xacro)
@@ -49,7 +49,7 @@
             <origin xyz = "0 -0.13 0" rpy="0 0 0" />
             <parent link="${prefix}palm" />
-            <child link="${prefix}vigir_gripper" />
-        </joint>
-        <link name="${prefix}vigir_gripper" />
+            <child link="${prefix}hand" />
+        </joint>
+        <link name="${prefix}hand" />
         <!-- thumb base -->
         <joint name="${prefix}thumb_roll" type="revolute">

Commit message: Switching hand -> palm ordering.

File: urdf/hdt_7dof_hand.xacro (robot description, xacro)
@@ -40,5 +40,5 @@
         <!-- gripper frame -->
         <joint name="${prefix}gripper_frame_joint" type="fixed">
-            <origin xyz="0 -0.13 0" rpy="0 0 -1.57079" />
+            <origin xyz="0 0 0" rpy="0 0 -1.57079" />
             <parent link="${prefix}palm" />
             <child link="${prefix}gripper_frame" />
@@ -47,7 +47,7 @@
         <!-- Hacked in joint to match ViGIR frames -->
         <joint name="${prefix}vigir_joint" type="fixed">
-            <origin xyz = "0 -0.13 0" rpy="0 0 0" />
-            <parent link="${prefix}palm" />
-            <child link="${prefix}hand" />
+            <origin xyz = "0 0.13 0" rpy="0 0 0" />
+            <parent link="${prefix}hand" />
+            <child link="${prefix}palm" />
         </joint>
         <link name="${prefix}hand" />

File: urdf/hdt_7dof_macro.xacro (robot description, xacro)
@@ -436,5 +436,5 @@
 			<origin xyz="0 -0.055 0" rpy="0 0 0"/>
 			<parent link="${prefix}wrist_yaw_bracket"/>
-			<child link="${prefix}palm"/>
+			<child link="${prefix}hand"/>
 		</joint>
 		<xacro:hdt_7dof_hand prefix="${prefix}" motor_base_id="${motor_base_id}" reflect="${reflect}" left_only="${left_only}" right_only="${right_only}" />

Commit message: fixed the dimensions to match that from our CAD data

File: urdf/hdt_7dof_hand.xacro (robot description, xacro)
@@ -102,5 +102,5 @@
             <axis xyz="1 0 0"/>
             <limit effort="4.0" lower="-0.7854" upper="1.5708" velocity="4.1888"/>
-            <origin xyz="0.00214 -0.02759 0.05700" rpy="0 0 0"/>
+            <origin xyz="0.00214 -0.030093 0.05703" rpy="0 0 0"/>
             <parent link="${prefix}thumb_base"/>
             <child link="${prefix}thumb_prox"/>
@@ -204,5 +204,5 @@
             <axis xyz="0 0 ${reflect*-1}"/>
             <limit effort="4.0" lower="${left_only*-1.5708 + right_only*-0.7854}" upper="${left_only*0.7854 + right_only*1.5708}" velocity="4.1888"/>
-            <origin xyz="0 -0.16325 0.02701" rpy="0 ${left_only*3.1416} 0"/>
+            <origin xyz="0 -0.163498 0.027" rpy="0 ${left_only*3.1416} 0"/>
             <parent link="${prefix}palm"/>
             <child link="${prefix}index_prox"/>
@@ -306,5 +306,5 @@
             <axis xyz="0 0 ${reflect*-1}"/>
             <limit effort="4.0" lower="${left_only*-1.5708 + right_only*-0.7854}" upper="${left_only*0.7854 + right_only*1.5708}" velocity="4.1888"/>
-            <origin xyz="0 -0.16325 -0.02701" rpy="0 ${left_only*3.1416} 0"/>
+            <origin xyz="0 -0.163498 -0.027" rpy="0 ${left_only*3.1416} 0"/>
             <parent link="${prefix}palm"/>
             <child link="${prefix}ring_prox"/>

File: urdf/hdt_7dof_hand_bbox.xacro (robot description, xacro)
@@ -96,5 +96,5 @@
             <axis xyz="1 0 0"/>
             <limit effort="4.0" lower="-0.7854" upper="1.5708" velocity="4.1888"/>
-            <origin xyz="0.00214 -0.02759 0.05700" rpy="0 0 0"/>
+            <origin xyz="0.002143 -0.030093 0.0573" rpy="0 0 0"/>
             <parent link="${prefix}thumb_base"/>
             <child link="${prefix}thumb_prox"/>
@@ -166,5 +166,5 @@
             <axis xyz="0 0 ${reflect*-1}"/>
             <limit effort="4.0" lower="${left_only*-1.5708 + right_only*-0.7854}" upper="${left_only*0.7854 + right_only*1.5708}" velocity="4.1888"/>
-            <origin xyz="0 -0.16325 0.02701" rpy="0 ${left_only*3.1416} 0"/>
+            <origin xyz="0 -0.163498 0.027" rpy="0 ${left_only*3.1416} 0"/>
             <parent link="${prefix}palm"/>
             <child link="${prefix}index_prox"/>
@@ -233,5 +233,5 @@
             <axis xyz="0 0 ${reflect*-1}"/>
             <limit effort="4.0" lower="${left_only*-1.5708 + right_only*-0.7854}" upper="${left_only*0.7854 + right_only*1.5708}" velocity="4.1888"/>
-            <origin xyz="0 -0.16325 -0.02701" rpy="0 ${left_only*3.1416} 0"/>
+            <origin xyz="0 -0.163498 -0.027" rpy="0 ${left_only*3.1416} 0"/>
             <parent link="${prefix}palm"/>
             <child link="${prefix}ring_prox"/>

File: urdf/hdt_7dof_macro.xacro (robot description, xacro)
@@ -72,5 +72,5 @@
 			<parent link="${prefix}shoulder"/>
 			<child link="${prefix}shoulder_roll_bracket"/>
-			<origin xyz="-0.09217 0 0" rpy="0 0 0"/>
+			<origin xyz="-0.093 0 0" rpy="0 0 0"/>
 		</joint>
 		<link name="${prefix}shoulder_roll_bracket">
@@ -191,5 +191,5 @@
 		</gazebo>
 		<joint name="${prefix}upper_arm_fixed" type="fixed">
-			<origin xyz="0 0 -0.16271" rpy="0 0 0"/>
+			<origin xyz="0 0 -0.1716" rpy="0 0 0"/>
 			<parent link="${prefix}upper_arm"/>
 			<child link="${prefix}elbow_pitch_bracket"/>
@@ -312,5 +312,5 @@
 		</gazebo>
 		<joint name="${prefix}forearm_fixed" type="fixed">
-			<origin xyz="0 -0.09217 0" rpy="0 0 0"/>
+			<origin xyz="0 -0.0751 0" rpy="0 0 0"/>
 			<parent link="${prefix}forearm"/>
 			<child link="${prefix}wrist_pitch_bracket"/>
@@ -392,5 +392,5 @@
 			<axis xyz="0 0 1"/>
 			<limit effort="60.0" lower="-1.5708" upper="1.5708" velocity="2.0944"/>
-			<origin xyz="0 -0.0771 0" rpy="0 0 0"/>
+			<origin xyz="0 -0.0741 0" rpy="0 0 0"/>
 			<parent link="${prefix}wrist_motors"/>
 			<child link="${prefix}wrist_yaw_bracket"/>

File: urdf/hdt_7dof_macro_bbox.xacro (robot description, xacro)
@@ -56,5 +56,5 @@
 			<parent link="${prefix}shoulder"/>
 			<child link="${prefix}shoulder_roll_bracket"/>
-			<origin xyz="-0.09217 0 0" rpy="0 0 0"/>
+			<origin xyz="-0.093 0 0" rpy="0 0 0"/>
 		</joint>
 		<link name="${prefix}shoulder_roll_bracket">
@@ -153,5 +153,5 @@
 		</link>
 		<joint name="${prefix}upper_arm_fixed" type="fixed">
-			<origin xyz="0 0 -0.16271" rpy="0 0 0"/>
+			<origin xyz="0 0 -0.1716" rpy="0 0 0"/>
 			<parent link="${prefix}upper_arm"/>
 			<child link="${prefix}elbow_pitch_bracket"/>
@@ -239,5 +239,5 @@
 		</link>
 		<joint name="${prefix}forearm_fixed" type="fixed">
-			<origin xyz="0 -0.09217 0" rpy="0 0 0"/>
+			<origin xyz="0 -0.0751 0" rpy="0 0 0"/>
 			<parent link="${prefix}forearm"/>
 			<child link="${prefix}wrist_pitch_bracket"/>
@@ -300,5 +300,5 @@
 			<axis xyz="0 0 1"/>
 			<limit effort="60.0" lower="-1.5708" upper="1.5708" velocity="2.0944"/>
-			<origin xyz="0 -0.0771 0" rpy="0 0 0"/>
+			<origin xyz="0 -0.0741 0" rpy="0 0 0"/>
 			<parent link="${prefix}wrist_motors"/>
 			<child link="${prefix}wrist_yaw_bracket"/>
