Commit message: updated the bounding boxes to completely match the sdf collision boxes and CAD stls

File: urdf/hdt_7dof_hand_bbox.xacro (robot description, xacro)
@@ -14,13 +14,13 @@
         <link name="${prefix}palm">
             <collision>
-                <origin xyz="0 -0.08 0" rpy="0 0 1.57079633"/>
-                <geometry>
-                    <box size="0.17 0.055 0.1"/>
-                </geometry>
-            </collision>
-            <visual>
-                <origin xyz="0 -0.08 0" rpy="0 0 1.57079633"/>
-                <geometry>
-                    <box size="0.17 0.055 0.1"/>
+                <origin xyz="0 -0.069749 0.005" rpy="0 0 1.57079633"/>
+                <geometry>
+                    <box size="0.18 0.071 0.105"/>
+                </geometry>
+            </collision>
+            <visual>
+                <origin xyz="0 -0.069749 0.005" rpy="0 0 1.57079633"/>
+                <geometry>
+                    <box size="0.18 0.071 0.105"/>
                 </geometry>
                 <material name="${prefix}black"/>
@@ -70,13 +70,13 @@
         <link name="${prefix}thumb_base">
             <collision>
-                <origin xyz="0 -0.025 0.0075" rpy="0 0 1.57079633"/>
-                <geometry>
-                    <box size="0.05 0.05 0.08"/>
-                </geometry>
-            </collision>
-            <visual>
-                <origin xyz="0 -0.025 0.0075" rpy="0 0 1.57079633"/>
-                <geometry>
-                    <box size="0.05 0.05 0.08"/>
+                <origin xyz="0 -0.03495 0.02903155" rpy="0 0 1.57079633"/>
+                <geometry>
+                    <box size="0.05 0.05 0.07"/>
+                </geometry>
+            </collision>
+            <visual>
+                <origin xyz="0 -0.03495 0.02903155" rpy="0 0 1.57079633"/>
+                <geometry>
+                    <box size="0.05 0.05 0.07"/>
                 </geometry>
                 <material name="${prefix}grey"/>
@@ -112,13 +112,13 @@
         <link name="${prefix}thumb_prox">
             <collision>
-                <origin xyz="0 0 0.05" rpy="0 0 0"/>
-                <geometry>
-                    <cylinder length="0.12" radius="0.02"/>
-                </geometry>
-            </collision>
-            <visual>
-                <origin xyz="0 0 0.05" rpy="0 0 0"/>
-                <geometry>
-                    <cylinder length="0.12" radius="0.02"/>
+                <origin xyz="0 -0.00154045 0.05414235" rpy="0 0 0"/>
+                <geometry>
+                    <cylinder length="0.10" radius="0.025"/>
+                </geometry>
+            </collision>
+            <visual>
+                <origin xyz="0 -0.00154045 0.05414235" rpy="0 0 0"/>
+                <geometry>
+                    <cylinder length="0.10" radius="0.025"/>
                 </geometry>
                 <material name="${prefix}grey"/>
@@ -182,13 +182,13 @@
         <link name="${prefix}index_prox">
             <collision>
-                <origin xyz="0 -0.05 0" rpy="-1.57079633 0 0"/>
-                <geometry>
-                    <cylinder length="0.12" radius="0.02"/>
-                </geometry>
-            </collision>
-            <visual>
-                <origin xyz="0 -0.05 0" rpy="-1.57079633 0 0"/>
-                <geometry>
-                    <cylinder length="0.12" radius="0.02"/>
+                <origin xyz="0.00154045 -0.04442185 0" rpy="-1.57079633 0 0"/>
+                <geometry>
+                    <cylinder length="0.10" radius="0.025"/>
+                </geometry>
+            </collision>
+            <visual>
+                <origin xyz="0.00154045 -0.04442185 0" rpy="-1.57079633 0 0"/>
+                <geometry>
+                    <cylinder length="0.10" radius="0.025"/>
                 </geometry>
                 <material name="${prefix}grey"/>
@@ -249,13 +249,13 @@
         <link name="${prefix}ring_prox">
             <collision>
-                <origin xyz="0 -0.05 0" rpy="-1.57079633 0 0"/>
-                <geometry>
-                    <cylinder length="0.12" radius="0.02"/>
-                </geometry>
-            </collision>
-            <visual>
-                <origin xyz="0 -0.05 0" rpy="-1.57079633 0 0"/>
-                <geometry>
-                    <cylinder length="0.12" radius="0.02"/>
+                <origin xyz="0.00154045 -0.04442185 0" rpy="-1.57079633 0 0"/>
+                <geometry>
+                    <cylinder length="0.10" radius="0.025"/>
+                </geometry>
+            </collision>
+            <visual>
+                <origin xyz="0.00154045 -0.04442185 0" rpy="-1.57079633 0 0"/>
+                <geometry>
+                    <cylinder length="0.10" radius="0.025"/>
                 </geometry>
                 <material name="${prefix}grey"/>

File: urdf/hdt_7dof_macro_bbox.xacro (robot description, xacro)
@@ -60,5 +60,5 @@
 		<link name="${prefix}shoulder_roll_bracket">
 			<collision>
-				<origin xyz="0 0 0" rpy="0 1.57079633 0"/>
+				<origin xyz="-0.009 0 0" rpy="0 1.57079633 0"/>
 				<geometry>
 				  <cylinder length="0.2" radius="0.05" />
@@ -66,5 +66,5 @@
 			</collision>
 			<visual>
-				<origin xyz="0 0 0" rpy="0 1.57079633 0"/>
+				<origin xyz="-0.009 0 0" rpy="0 1.57079633 0"/>
 				<geometry>
 					<cylinder length="0.2" radius="0.05" />
@@ -102,5 +102,5 @@
 		<link name="${prefix}shoulder_roll_motor">
 			<collision>
-				<origin xyz="0 0 -0.16" rpy="0 0 0"/>
+				<origin xyz="0 0 -0.2183" rpy="0 0 0"/>
 				<geometry>
 					<cylinder length="0.32" radius="0.05"/>
@@ -108,5 +108,5 @@
 			</collision>
 			<visual>
-				<origin xyz="0 0 -0.16" rpy="0 0 0"/>
+				<origin xyz="0 0 -0.2183" rpy="0 0 0"/>
 				<geometry>
 					<cylinder length="0.32" radius="0.05"/>
@@ -188,13 +188,13 @@
 		<link name="${prefix}elbow_pitch_motor">
 			<collision>
-				<origin xyz="0 -0.1 0" rpy="1.57079633 0 0"/>
-				<geometry>
-					<cylinder length="0.2" radius="0.05"/>
-				</geometry>
-			</collision>
-			<visual>
-				<origin xyz="0 -0.1 0" rpy="1.57079633 0 0"/>
-				<geometry>
-					<cylinder length="0.2" radius="0.05"/>
+				<origin xyz="0 -0.1126 0" rpy="1.57079633 0 0"/>
+				<geometry>
+					<cylinder length="0.1" radius="0.05"/>
+				</geometry>
+			</collision>
+			<visual>
+				<origin xyz="0 -0.1126 0" rpy="1.57079633 0 0"/>
+				<geometry>
+					<cylinder length="0.1" radius="0.05"/>
 				</geometry>
 				<material name="${prefix}green"/>
