Commit message: Rename links to be more descriptive

File: urdf/hdt_7dof_macro.xacro (robot description, xacro)
@@ -39,5 +39,5 @@
 			<origin xyz="${x} ${y} ${z}" rpy="0 0 ${yaw}"/>
 			<parent link="${parent}"/>
-			<child link="${prefix}link1"/>
+			<child link="${prefix}shoulder"/>
 			<dynamics damping="0.7" friction="0.0"/>
 		</joint>
@@ -51,5 +51,5 @@
 			</actuator>
 		</transmission>
-		<link name="${prefix}link1">
+		<link name="${prefix}shoulder">
 			<collision>
 				<origin xyz="0 0 0" rpy="0 0 0"/>
@@ -74,13 +74,13 @@
 			</inertial>
 		</link>
-		<gazebo reference="${prefix}link1">
+		<gazebo reference="${prefix}shoulder">
 			<material>Gazebo/Green</material>
 		</gazebo>
-		<joint name="${prefix}joint1f" type="fixed">
-			<parent link="${prefix}link1"/>
-			<child link="${prefix}link2a"/>
+		<joint name="${prefix}shoulder_fixed" type="fixed">
+			<parent link="${prefix}shoulder"/>
+			<child link="${prefix}shoulder_roll_bracket"/>
 			<origin xyz="-0.09217 0 0" rpy="0 0 0"/>
 		</joint>
-		<link name="${prefix}link2a">
+		<link name="${prefix}shoulder_roll_bracket">
 			<collision>
 				<origin xyz="0 0 0" rpy="0 0 0"/>
@@ -105,5 +105,5 @@
 			</inertial>
 		</link>
-		<gazebo reference="${prefix}link2a">
+		<gazebo reference="${prefix}shoulder_roll_bracket">
 			<material>Gazebo/Black</material>
 		</gazebo>
@@ -114,6 +114,6 @@
 			<limit effort="60.0" lower="${left_only*-0.5236 + right_only*-3.1416}" upper="${left_only*3.1416 + right_only*0.5236}" velocity="2.0944"/>
 			<origin xyz="-0.07 0 0" rpy="0 0 0"/>
-			<parent link="${prefix}link2a"/>
-			<child link="${prefix}link2b"/>
+			<parent link="${prefix}shoulder_roll_bracket"/>
+			<child link="${prefix}shoulder_roll_motor"/>
 			<dynamics damping="0.7" friction="0.0"/>
 		</joint>
@@ -127,5 +127,5 @@
 			</actuator>
 		</transmission>
-		<link name="${prefix}link2b">
+		<link name="${prefix}shoulder_roll_motor">
 			<collision>
 				<origin xyz="0 0 0" rpy="0 0 0"/>
@@ -150,5 +150,5 @@
 			</inertial>
 		</link>
-		<gazebo reference="${prefix}link2b">
+		<gazebo reference="${prefix}shoulder_roll_motor">
 			<material>Gazebo/Grey</material>
 		</gazebo>
@@ -159,6 +159,6 @@
 			<limit effort="60.0" lower="-2.0944" upper="2.0944" velocity="2.0944"/>
 			<origin xyz="0 0 -0.077" rpy="0 0 0" />
-			<parent link="${prefix}link2b"/>
-			<child link="${prefix}link3"/>
+			<parent link="${prefix}shoulder_roll_motor"/>
+			<child link="${prefix}upper_arm"/>
 			<dynamics damping="0.7" friction="0.0"/>
 		</joint>
@@ -172,5 +172,5 @@
 			</actuator>
 		</transmission>
-		<link name="${prefix}link3">
+		<link name="${prefix}upper_arm">
 			<collision>
 				<origin xyz="0 0 0.0" rpy="0 0 0"/>
@@ -195,13 +195,13 @@
 			</inertial>
 		</link>
-		<gazebo reference="${prefix}link3">
+		<gazebo reference="${prefix}upper_arm">
 			<material>Gazebo/Green</material>
 		</gazebo>
-		<joint name="${prefix}joint3f" type="fixed">
+		<joint name="${prefix}upper_arm_fixed" type="fixed">
 			<origin xyz="0 0 -0.16271" rpy="0 0 0"/>
-			<parent link="${prefix}link3"/>
-			<child link="${prefix}link4a"/>
-		</joint>
-		<link name="${prefix}link4a">
+			<parent link="${prefix}upper_arm"/>
+			<child link="${prefix}elbow_pitch_bracket"/>
+		</joint>
+		<link name="${prefix}elbow_pitch_bracket">
 			<collision>
 				<origin xyz="0 0 0" rpy="0 0 0"/>
@@ -226,5 +226,5 @@
 			</inertial>
 		</link>
-		<gazebo reference="${prefix}link4a">
+		<gazebo reference="${prefix}elbow_pitch_bracket">
 			<material>Gazebo/Black</material>
 		</gazebo>
@@ -235,6 +235,6 @@
 			<limit effort="60.0" lower="-0.5236" upper="3.6652" velocity="2.0944"/>
 			<origin xyz="0 0 -0.07" rpy="${left_only*3.1416} 0 0"/>
-			<parent link="${prefix}link4a"/>
-			<child link="${prefix}link4b"/>
+			<parent link="${prefix}elbow_pitch_bracket"/>
+			<child link="${prefix}elbow_pitch_motor"/>
 			<dynamics damping="0.7" friction="0.0"/>
 		</joint>
@@ -248,5 +248,5 @@
 			</actuator>
 		</transmission>
-		<link name="${prefix}link4b">
+		<link name="${prefix}elbow_pitch_motor">
 			<collision>
 				<origin xyz="0 0 0" rpy="0 0 0"/>
@@ -271,5 +271,5 @@
 			</inertial>
 		</link>
-		<gazebo reference="${prefix}link4b">
+		<gazebo reference="${prefix}elbow_pitch_motor">
 			<material>Gazebo/Grey</material>
 		</gazebo>
@@ -280,6 +280,6 @@
 			<limit effort="60.0" lower="-2.0944" upper="2.0944" velocity="2.0944"/>
 			<origin xyz="0 -0.077 0" rpy="0 ${left_only*3.1416} 0"/>
-			<parent link="${prefix}link4b"/>
-			<child link="${prefix}link5"/>
+			<parent link="${prefix}elbow_pitch_motor"/>
+			<child link="${prefix}forearm"/>
 			<dynamics damping="0.7" friction="0.0"/>
 		</joint>
@@ -293,5 +293,5 @@
 			</actuator>
 		</transmission>
-		<link name="${prefix}link5">
+		<link name="${prefix}forearm">
 			<collision>
 				<origin xyz="0 0 0.0" rpy="0 0 0"/>
@@ -316,13 +316,13 @@
 			</inertial>
 		</link>
-		<gazebo reference="${prefix}link5">
+		<gazebo reference="${prefix}forearm">
 			<material>Gazebo/Green</material>
 		</gazebo>
-		<joint name="${prefix}joint5f" type="fixed">
+		<joint name="${prefix}forearm_fixed" type="fixed">
 			<origin xyz="0 -0.09217 0" rpy="0 0 0"/>
-			<parent link="${prefix}link5"/>
-			<child link="${prefix}link6a"/>
-		</joint>
-		<link name="${prefix}link6a">
+			<parent link="${prefix}forearm"/>
+			<child link="${prefix}wrist_pitch_bracket"/>
+		</joint>
+		<link name="${prefix}wrist_pitch_bracket">
 			<collision>
 				<origin xyz="0 0 0" rpy="0 0 0"/>
@@ -347,5 +347,5 @@
 			</inertial>
 		</link>
-		<gazebo reference="${prefix}link6a">
+		<gazebo reference="${prefix}wrist_pitch_bracket">
 			<material>Gazebo/Black</material>
 		</gazebo>
@@ -356,6 +356,6 @@
 			<limit effort="60.0" lower="-1.5708" upper="1.5708" velocity="2.0944"/>
 			<origin xyz="0 -0.055 0" rpy="0 0 0"/>
-			<parent link="${prefix}link6a"/>
-			<child link="${prefix}link6b"/>
+			<parent link="${prefix}wrist_pitch_bracket"/>
+			<child link="${prefix}wrist_motors"/>
 			<dynamics damping="0.7" friction="0.0"/>
 		</joint>
@@ -369,5 +369,5 @@
 			</actuator>
 		</transmission>
-		<link name="${prefix}link6b">
+		<link name="${prefix}wrist_motors">
 			<collision>
 				<origin xyz="0 0 0" rpy="0 0 0"/>
@@ -392,5 +392,5 @@
 			</inertial>
 		</link>
-		<gazebo reference="${prefix}link6b">
+		<gazebo reference="${prefix}wrist_motors">
 			<material>Gazebo/Grey</material>
 		</gazebo>
@@ -401,6 +401,6 @@
 			<limit effort="60.0" lower="-1.5708" upper="1.5708" velocity="2.0944"/>
 			<origin xyz="0 -0.0771 0" rpy="0 0 0"/>
-			<parent link="${prefix}link6b"/>
-			<child link="${prefix}link7"/>
+			<parent link="${prefix}wrist_motors"/>
+			<child link="${prefix}wrist_yaw_bracket"/>
 			<dynamics damping="0.7" friction="0.0"/>
 		</joint>
@@ -414,5 +414,5 @@
 			</actuator>
 		</transmission>
-		<link name="${prefix}link7">
+		<link name="${prefix}wrist_yaw_bracket">
 			<collision>
 				<origin xyz="0 0 0" rpy="0 0 0"/>
@@ -437,5 +437,5 @@
 			</inertial>
 		</link>
-		<gazebo reference="${prefix}link7">
+		<gazebo reference="${prefix}wrist_yaw_bracket">
 			<material>Gazebo/Black</material>
 		</gazebo>
@@ -443,5 +443,5 @@
 		<joint name="${prefix}palm" type="fixed">
 			<origin xyz="0 -0.055 0" rpy="0 0 0"/>
-			<parent link="${prefix}link7"/>
+			<parent link="${prefix}wrist_yaw_bracket"/>
 			<child link="${prefix}palm"/>
 		</joint>

Commit message: Rename STLs to match links
Also consolidates the finger STLs, which were identical.

File: urdf/hdt_7dof_macro.xacro (robot description, xacro)
@@ -55,11 +55,11 @@
 				<origin xyz="0 0 0" rpy="0 0 0"/>
 				<geometry>
-					<mesh filename="package://hdt_7dof_description/meshes/hdt_7dof_1_right.STL"/>
-				</geometry>
-			</collision>
-			<visual>
-				<origin xyz="0 0 0" rpy="0 0 0"/>
-				<geometry>
-					<mesh filename="package://hdt_7dof_description/meshes/hdt_7dof_1_right.STL"/>
+					<mesh filename="package://hdt_7dof_description/meshes/shoulder.stl"/>
+				</geometry>
+			</collision>
+			<visual>
+				<origin xyz="0 0 0" rpy="0 0 0"/>
+				<geometry>
+					<mesh filename="package://hdt_7dof_description/meshes/shoulder.stl"/>
 				</geometry>
 				<material name="${prefix}green"/>
@@ -86,11 +86,11 @@
 				<origin xyz="0 0 0" rpy="0 0 0"/>
 				<geometry>
-					<mesh filename="package://hdt_7dof_description/meshes/hdt_7dof_2a_right.STL"/>
-				</geometry>
-			</collision>
-			<visual>
-				<origin xyz="0 0 0" rpy="0 0 0"/>
-				<geometry>
-					<mesh filename="package://hdt_7dof_description/meshes/hdt_7dof_2a_right.STL"/>
+					<mesh filename="package://hdt_7dof_description/meshes/shoulder_roll_bracket.stl"/>
+				</geometry>
+			</collision>
+			<visual>
+				<origin xyz="0 0 0" rpy="0 0 0"/>
+				<geometry>
+					<mesh filename="package://hdt_7dof_description/meshes/shoulder_roll_bracket.stl"/>
 				</geometry>
 				<material name="${prefix}black"/>
@@ -131,11 +131,11 @@
 				<origin xyz="0 0 0" rpy="0 0 0"/>
 				<geometry>
-					<mesh filename="package://hdt_7dof_description/meshes/hdt_7dof_2b.STL"/>
-				</geometry>
-			</collision>
-			<visual>
-				<origin xyz="0 0 0.0" rpy="0 0 0"/>
-				<geometry>
-					<mesh filename="package://hdt_7dof_description/meshes/hdt_7dof_2b.STL"/>
+					<mesh filename="package://hdt_7dof_description/meshes/shoulder_roll_motor.stl"/>
+				</geometry>
+			</collision>
+			<visual>
+				<origin xyz="0 0 0.0" rpy="0 0 0"/>
+				<geometry>
+					<mesh filename="package://hdt_7dof_description/meshes/shoulder_roll_motor.stl"/>
 				</geometry>
 				<material name="${prefix}grey"/>
@@ -176,11 +176,11 @@
 				<origin xyz="0 0 0.0" rpy="0 0 0"/>
 				<geometry>
-					<mesh filename="package://hdt_7dof_description/meshes/hdt_7dof_3.STL"/>
-				</geometry>
-			</collision>
-			<visual>
-				<origin xyz="0 0 0.0" rpy="0 0 0"/>
-				<geometry>
-					<mesh filename="package://hdt_7dof_description/meshes/hdt_7dof_3.STL"/>
+					<mesh filename="package://hdt_7dof_description/meshes/upper_arm.stl"/>
+				</geometry>
+			</collision>
+			<visual>
+				<origin xyz="0 0 0.0" rpy="0 0 0"/>
+				<geometry>
+					<mesh filename="package://hdt_7dof_description/meshes/upper_arm.stl"/>
 				</geometry>
 				<material name="${prefix}green"/>
@@ -207,11 +207,11 @@
 				<origin xyz="0 0 0" rpy="0 0 0"/>
 				<geometry>
-					<mesh filename="package://hdt_7dof_description/meshes/hdt_7dof_4a.STL"/>
-				</geometry>
-			</collision>
-			<visual>
-				<origin xyz="0 0 0.0" rpy="0 0 0"/>
-				<geometry>
-					<mesh filename="package://hdt_7dof_description/meshes/hdt_7dof_4a.STL"/>
+					<mesh filename="package://hdt_7dof_description/meshes/elbow_pitch_bracket.stl"/>
+				</geometry>
+			</collision>
+			<visual>
+				<origin xyz="0 0 0.0" rpy="0 0 0"/>
+				<geometry>
+					<mesh filename="package://hdt_7dof_description/meshes/elbow_pitch_bracket.stl"/>
 				</geometry>
 				<material name="${prefix}black"/>
@@ -252,11 +252,11 @@
 				<origin xyz="0 0 0" rpy="0 0 0"/>
 				<geometry>
-					<mesh filename="package://hdt_7dof_description/meshes/hdt_7dof_4b.STL"/>
-				</geometry>
-			</collision>
-			<visual>
-				<origin xyz="0 0 0.0" rpy="0 0 0"/>
-				<geometry>
-					<mesh filename="package://hdt_7dof_description/meshes/hdt_7dof_4b.STL"/>
+					<mesh filename="package://hdt_7dof_description/meshes/elbow_pitch_motor.stl"/>
+				</geometry>
+			</collision>
+			<visual>
+				<origin xyz="0 0 0.0" rpy="0 0 0"/>
+				<geometry>
+					<mesh filename="package://hdt_7dof_description/meshes/elbow_pitch_motor.stl"/>
 				</geometry>
 				<material name="${prefix}grey"/>
@@ -297,11 +297,11 @@
 				<origin xyz="0 0 0.0" rpy="0 0 0"/>
 				<geometry>
-					<mesh filename="package://hdt_7dof_description/meshes/hdt_7dof_5.STL"/>
-				</geometry>
-			</collision>
-			<visual>
-				<origin xyz="0 0 0.0" rpy="0 0 0"/>
-				<geometry>
-					<mesh filename="package://hdt_7dof_description/meshes/hdt_7dof_5.STL"/>
+					<mesh filename="package://hdt_7dof_description/meshes/forearm.stl"/>
+				</geometry>
+			</collision>
+			<visual>
+				<origin xyz="0 0 0.0" rpy="0 0 0"/>
+				<geometry>
+					<mesh filename="package://hdt_7dof_description/meshes/forearm.stl"/>
 				</geometry>
 				<material name="${prefix}green"/>
@@ -328,11 +328,11 @@
 				<origin xyz="0 0 0" rpy="0 0 0"/>
 				<geometry>
-					<mesh filename="package://hdt_7dof_description/meshes/hdt_7dof_6a.STL"/>
-				</geometry>
-			</collision>
-			<visual>
-				<origin xyz="0 0 0.0" rpy="0 0 0"/>
-				<geometry>
-					<mesh filename="package://hdt_7dof_description/meshes/hdt_7dof_6a.STL"/>
+					<mesh filename="package://hdt_7dof_description/meshes/wrist_pitch_bracket.stl"/>
+				</geometry>
+			</collision>
+			<visual>
+				<origin xyz="0 0 0.0" rpy="0 0 0"/>
+				<geometry>
+					<mesh filename="package://hdt_7dof_description/meshes/wrist_pitch_bracket.stl"/>
 				</geometry>
 				<material name="${prefix}black"/>
@@ -373,11 +373,11 @@
 				<origin xyz="0 0 0" rpy="0 0 0"/>
 				<geometry>
-					<mesh filename="package://hdt_7dof_description/meshes/hdt_7dof_6b.STL"/>
-				</geometry>
-			</collision>
-			<visual>
-				<origin xyz="0 0 0.0" rpy="0 0 0"/>
-				<geometry>
-					<mesh filename="package://hdt_7dof_description/meshes/hdt_7dof_6b.STL"/>
+					<mesh filename="package://hdt_7dof_description/meshes/wrist_motors.stl"/>
+				</geometry>
+			</collision>
+			<visual>
+				<origin xyz="0 0 0.0" rpy="0 0 0"/>
+				<geometry>
+					<mesh filename="package://hdt_7dof_description/meshes/wrist_motors.stl"/>
 				</geometry>
 				<material name="${prefix}grey"/>
@@ -418,11 +418,11 @@
 				<origin xyz="0 0 0" rpy="0 0 0"/>
 				<geometry>
-					<mesh filename="package://hdt_7dof_description/meshes/hdt_7dof_7.STL"/>
-				</geometry>
-			</collision>
-			<visual>
-				<origin xyz="0 0 0.0" rpy="0 0 0"/>
-				<geometry>
-					<mesh filename="package://hdt_7dof_description/meshes/hdt_7dof_7.STL"/>
+					<mesh filename="package://hdt_7dof_description/meshes/wrist_yaw_bracket.stl"/>
+				</geometry>
+			</collision>
+			<visual>
+				<origin xyz="0 0 0.0" rpy="0 0 0"/>
+				<geometry>
+					<mesh filename="package://hdt_7dof_description/meshes/wrist_yaw_bracket.stl"/>
 				</geometry>
 				<material name="${prefix}black"/>
@@ -450,11 +450,11 @@
 				<origin xyz="0 0 0" rpy="0 0 0"/>
 				<geometry>
-					<mesh filename="package://hdt_7dof_description/meshes/hdt_7dof_palm.STL"/>
-				</geometry>
-			</collision>
-			<visual>
-				<origin xyz="0 0 0.0" rpy="0 0 0"/>
-				<geometry>
-					<mesh filename="package://hdt_7dof_description/meshes/hdt_7dof_palm.STL"/>
+					<mesh filename="package://hdt_7dof_description/meshes/palm.stl"/>
+				</geometry>
+			</collision>
+			<visual>
+				<origin xyz="0 0 0.0" rpy="0 0 0"/>
+				<geometry>
+					<mesh filename="package://hdt_7dof_description/meshes/palm.stl"/>
 				</geometry>
 				<material name="${prefix}black"/>
@@ -502,11 +502,11 @@
 				<origin xyz="0 0 0" rpy="0 0 0"/>
 				<geometry>
-					<mesh filename="package://hdt_7dof_description/meshes/hdt_7dof_thumb_base.STL"/>
-				</geometry>
-			</collision>
-			<visual>
-				<origin xyz="0 0 0" rpy="0 0 0"/>
-				<geometry>
-					<mesh filename="package://hdt_7dof_description/meshes/hdt_7dof_thumb_base.STL"/>
+					<mesh filename="package://hdt_7dof_description/meshes/thumb_base.stl"/>
+				</geometry>
+			</collision>
+			<visual>
+				<origin xyz="0 0 0" rpy="0 0 0"/>
+				<geometry>
+					<mesh filename="package://hdt_7dof_description/meshes/thumb_base.stl"/>
 				</geometry>
 				<material name="${prefix}grey"/>
@@ -547,11 +547,11 @@
 				<origin xyz="0 0 0" rpy="0 0 0"/>
 				<geometry>
-					<mesh filename="package://hdt_7dof_description/meshes/hdt_7dof_thumb_prox.STL"/>
-				</geometry>
-			</collision>
-			<visual>
-				<origin xyz="0 0 0" rpy="0 0 0"/>
-				<geometry>
-					<mesh filename="package://hdt_7dof_description/meshes/hdt_7dof_thumb_prox.STL"/>
+					<mesh filename="package://hdt_7dof_description/meshes/thumb_prox.stl"/>
+				</geometry>
+			</collision>
+			<visual>
+				<origin xyz="0 0 0" rpy="0 0 0"/>
+				<geometry>
+					<mesh filename="package://hdt_7dof_description/meshes/thumb_prox.stl"/>
 				</geometry>
 				<material name="${prefix}grey"/>
@@ -572,11 +572,11 @@
 				<origin xyz="0 0 0" rpy="0 0 0"/>
 				<geometry>
-					<mesh filename="package://hdt_7dof_description/meshes/hdt_7dof_thumb_med.STL"/>
-				</geometry>
-			</collision>
-			<visual>
-				<origin xyz="0 0 0" rpy="0 0 0"/>
-				<geometry>
-					<mesh filename="package://hdt_7dof_description/meshes/hdt_7dof_thumb_med.STL"/>
+					<mesh filename="package://hdt_7dof_description/meshes/thumb_med.stl"/>
+				</geometry>
+			</collision>
+			<visual>
+				<origin xyz="0 0 0" rpy="0 0 0"/>
+				<geometry>
+					<mesh filename="package://hdt_7dof_description/meshes/thumb_med.stl"/>
 				</geometry>
 				<material name="${prefix}black"/>
@@ -604,11 +604,11 @@
 				<origin xyz="0 0 0" rpy="0 0 0"/>
 				<geometry>
-					<mesh filename="package://hdt_7dof_description/meshes/hdt_7dof_thumb_dist.STL"/>
-				</geometry>
-			</collision>
-			<visual>
-				<origin xyz="0 0 0" rpy="0 0 0"/>
-				<geometry>
-					<mesh filename="package://hdt_7dof_description/meshes/hdt_7dof_thumb_dist.STL"/>
+					<mesh filename="package://hdt_7dof_description/meshes/thumb_dist.stl"/>
+				</geometry>
+			</collision>
+			<visual>
+				<origin xyz="0 0 0" rpy="0 0 0"/>
+				<geometry>
+					<mesh filename="package://hdt_7dof_description/meshes/thumb_dist.stl"/>
 				</geometry>
 				<material name="${prefix}grey"/>
@@ -649,11 +649,11 @@
 				<origin xyz="0 0 0" rpy="0 0 0"/>
 				<geometry>
-					<mesh filename="package://hdt_7dof_description/meshes/hdt_7dof_index_prox_right.STL"/>
-				</geometry>
-			</collision>
-			<visual>
-				<origin xyz="0 0 0" rpy="0 0 0"/>
-				<geometry>
-					<mesh filename="package://hdt_7dof_description/meshes/hdt_7dof_index_prox_right.STL"/>
+					<mesh filename="package://hdt_7dof_description/meshes/finger_prox_right.stl"/>
+				</geometry>
+			</collision>
+			<visual>
+				<origin xyz="0 0 0" rpy="0 0 0"/>
+				<geometry>
+					<mesh filename="package://hdt_7dof_description/meshes/finger_prox_right.stl"/>
 				</geometry>
 				<material name="${prefix}grey"/>
@@ -674,11 +674,11 @@
 				<origin xyz="0 0 0" rpy="0 0 0"/>
 				<geometry>
-					<mesh filename="package://hdt_7dof_description/meshes/hdt_7dof_index_med_right.STL"/>
-				</geometry>
-			</collision>
-			<visual>
-				<origin xyz="0 0 0" rpy="0 0 0"/>
-				<geometry>
-					<mesh filename="package://hdt_7dof_description/meshes/hdt_7dof_index_med_right.STL"/>
+					<mesh filename="package://hdt_7dof_description/meshes/finger_med_right.stl"/>
+				</geometry>
+			</collision>
+			<visual>
+				<origin xyz="0 0 0" rpy="0 0 0"/>
+				<geometry>
+					<mesh filename="package://hdt_7dof_description/meshes/finger_med_right.stl"/>
 				</geometry>
 				<material name="${prefix}black"/>
@@ -706,11 +706,11 @@
 				<origin xyz="0 0 0" rpy="0 0 0"/>
 				<geometry>
-					<mesh filename="package://hdt_7dof_description/meshes/hdt_7dof_index_dist_right.STL"/>
-				</geometry>
-			</collision>
-			<visual>
-				<origin xyz="0 0 0" rpy="0 0 0"/>
-				<geometry>
-					<mesh filename="package://hdt_7dof_description/meshes/hdt_7dof_index_dist_right.STL"/>
+					<mesh filename="package://hdt_7dof_description/meshes/finger_dist_right.stl"/>
+				</geometry>
+			</collision>
+			<visual>
+				<origin xyz="0 0 0" rpy="0 0 0"/>
+				<geometry>
+					<mesh filename="package://hdt_7dof_description/meshes/finger_dist_right.stl"/>
 				</geometry>
 				<material name="${prefix}grey"/>
@@ -751,11 +751,11 @@
 				<origin xyz="0 0 0" rpy="0 0 0"/>
 				<geometry>
-					<mesh filename="package://hdt_7dof_description/meshes/hdt_7dof_ring_prox_right.STL"/>
-				</geometry>
-			</collision>
-			<visual>
-				<origin xyz="0 0 0" rpy="0 0 0"/>
-				<geometry>
-					<mesh filename="package://hdt_7dof_description/meshes/hdt_7dof_ring_prox_right.STL"/>
+					<mesh filename="package://hdt_7dof_description/meshes/finger_prox_right.stl"/>
+				</geometry>
+			</collision>
+			<visual>
+				<origin xyz="0 0 0" rpy="0 0 0"/>
+				<geometry>
+					<mesh filename="package://hdt_7dof_description/meshes/finger_prox_right.stl"/>
 				</geometry>
 				<material name="${prefix}grey"/>
@@ -776,11 +776,11 @@
 				<origin xyz="0 0 0" rpy="0 0 0"/>
 				<geometry>
-					<mesh filename="package://hdt_7dof_description/meshes/hdt_7dof_ring_med_right.STL"/>
-				</geometry>
-			</collision>
-			<visual>
-				<origin xyz="0 0 0" rpy="0 0 0"/>
-				<geometry>
-					<mesh filename="package://hdt_7dof_description/meshes/hdt_7dof_ring_med_right.STL"/>
+					<mesh filename="package://hdt_7dof_description/meshes/finger_med_right.stl"/>
+				</geometry>
+			</collision>
+			<visual>
+				<origin xyz="0 0 0" rpy="0 0 0"/>
+				<geometry>
+					<mesh filename="package://hdt_7dof_description/meshes/finger_med_right.stl"/>
 				</geometry>
 				<material name="${prefix}black"/>
@@ -808,11 +808,11 @@
 				<origin xyz="0 0 0" rpy="0 0 0"/>
 				<geometry>
-					<mesh filename="package://hdt_7dof_description/meshes/hdt_7dof_ring_dist_right.STL"/>
-				</geometry>
-			</collision>
-			<visual>
-				<origin xyz="0 0 0" rpy="0 0 0"/>
-				<geometry>
-					<mesh filename="package://hdt_7dof_description/meshes/hdt_7dof_ring_dist_right.STL"/>
+					<mesh filename="package://hdt_7dof_description/meshes/finger_dist_right.stl"/>
+				</geometry>
+			</collision>
+			<visual>
+				<origin xyz="0 0 0" rpy="0 0 0"/>
+				<geometry>
+					<mesh filename="package://hdt_7dof_description/meshes/finger_dist_right.stl"/>
 				</geometry>
 				<material name="${prefix}grey"/>
