Commit message: Add hands as separate xacros for MoveIt.

File: urdf/hdt_7dof_macro.xacro (robot description, xacro)
@@ -7,14 +7,6 @@
 		<xacro:hdt_7dof reflect="-1" left_only="0" right_only="1" prefix="${prefix}" parent="${parent}" x="${x}" y="${y}" z="${z}" yaw="1.57079" motor_base_id="${motor_base_id}"/>
 	</xacro:macro>
-	<!-- default inertia -->
-	<xacro:macro name="default_inertial">
-		<inertial>
-			<mass value="0.025"/>
-			<inertia
-				ixx="0.0005" ixy="0.0" ixz="0.0"
-				iyy="0.0005" iyz="0.0"
-				izz="0.0005"/>
-		</inertial>
-	</xacro:macro>
+	<!-- hand included here -->
+	<xacro:include filename="$(find hdt_7dof_description)/urdf/hdt_7dof_hand.xacro" />
 	<!-- reflect: should be either 1 or -1, and can be multiplied to negate a side -->
 	<!--          the left:1, right:-1 mapping is the same as for PR2 (and works with the standard y axis) -->
@@ -446,388 +438,5 @@
 			<child link="${prefix}palm"/>
 		</joint>
-		<link name="${prefix}palm">
-			<collision>
-				<origin xyz="0 0 0" rpy="0 0 0"/>
-				<geometry>
-					<mesh filename="package://hdt_7dof_description/meshes/palm.stl"/>
-				</geometry>
-			</collision>
-			<visual>
-				<origin xyz="0 0 0.0" rpy="0 0 0"/>
-				<geometry>
-					<mesh filename="package://hdt_7dof_description/meshes/palm.stl"/>
-				</geometry>
-				<material name="${prefix}black"/>
-			</visual>
-			<inertial>
-				<origin xyz="0 -0.08326 -0.00539" rpy="0 0 0"/>
-				<mass value="0.56756"/>
-				<inertia
-					ixx="0.001727803" ixy="0.000001205" ixz="0.0"
-					iyy="0.000549457" iyz="-0.000101997"
-					izz="0.001418031"/>
-			</inertial>
-		</link>
-		<gazebo reference="${prefix}palm">
-			<material>Gazebo/Black</material>
-		</gazebo>
-		<!-- gripper frame -->
-		<joint name="${prefix}gripper_frame_joint" type="fixed">
-			<origin xyz="0 -0.13 0" rpy="0 0 -1.57079" />
-			<parent link="${prefix}palm" />
-			<child link="${prefix}gripper_frame" />
-		</joint>
-		<link name="${prefix}gripper_frame" />
-		<!-- thumb base -->
-		<joint name="${prefix}thumb_roll" type="revolute">
-			<hdt id="${motor_base_id + 9}" kmin="5" kmax="20" inertia="0.01"/>
-			<axis xyz="0 -1 0"/>
-			<limit effort="4.0" lower="-1.5708" upper="1.5708" velocity="4.1888"/>
-			<origin xyz="0 -0.05039 0.01529" rpy="0 0 0"/>
-			<parent link="${prefix}palm"/>
-			<child link="${prefix}thumb_base"/>
-			<dynamics damping="0.7" friction="0.0"/>
-		</joint>
-		<transmission name="${prefix}tran10">
-			<type>transmission_interface/SimpleTransmission</type>
-			<joint name="${prefix}thumb_roll">
-			</joint>
-			<actuator name="${prefix}motor10">
-				<hardwareInterface>EffortJointInterface</hardwareInterface>
-				<mechanicalReduction>1</mechanicalReduction>
-			</actuator>
-		</transmission>
-		<link name="${prefix}thumb_base">
-			<collision>
-				<origin xyz="0 0 0" rpy="0 0 0"/>
-				<geometry>
-					<mesh filename="package://hdt_7dof_description/meshes/thumb_base.stl"/>
-				</geometry>
-			</collision>
-			<visual>
-				<origin xyz="0 0 0" rpy="0 0 0"/>
-				<geometry>
-					<mesh filename="package://hdt_7dof_description/meshes/thumb_base.stl"/>
-				</geometry>
-				<material name="${prefix}grey"/>
-			</visual>
-			<inertial>
-				<origin xyz="0 -0.02653 0.02207" rpy="0 0 0"/>
-				<mass value="0.08562"/>
-				<inertia
-					ixx="0.0000315" ixy="0.0" ixz="0.0"
-					iyy="0.000034299" iyz="0.0"
-					izz="0.000022344"/>
-			</inertial>
-		</link>
-		<gazebo reference="${prefix}thumb_base">
-			<material>Gazebo/Grey</material>
-		</gazebo>
-		<!-- thumb prox -->
-		<joint name="${prefix}thumb_pitch" type="revolute">
-			<hdt id="${motor_base_id + 10}" kmin="5" kmax="20" inertia="0.01"/>
-			<axis xyz="1 0 0"/>
-			<limit effort="4.0" lower="-0.7854" upper="1.5708" velocity="4.1888"/>
-			<origin xyz="0.00214 -0.02759 0.05700" rpy="0 0 0"/>
-			<parent link="${prefix}thumb_base"/>
-			<child link="${prefix}thumb_prox"/>
-			<dynamics damping="0.7" friction="0.0"/>
-		</joint>
-		<transmission name="${prefix}tran11">
-			<type>transmission_interface/SimpleTransmission</type>
-			<joint name="${prefix}thumb_pitch">
-			</joint>
-			<actuator name="${prefix}motor11">
-				<hardwareInterface>EffortJointInterface</hardwareInterface>
-				<mechanicalReduction>1</mechanicalReduction>
-			</actuator>
-		</transmission>
-		<link name="${prefix}thumb_prox">
-			<collision>
-				<origin xyz="0 0 0" rpy="0 0 0"/>
-				<geometry>
-					<mesh filename="package://hdt_7dof_description/meshes/thumb_prox.stl"/>
-				</geometry>
-			</collision>
-			<visual>
-				<origin xyz="0 0 0" rpy="0 0 0"/>
-				<geometry>
-					<mesh filename="package://hdt_7dof_description/meshes/thumb_prox.stl"/>
-				</geometry>
-				<material name="${prefix}grey"/>
-			</visual>
-			<xacro:default_inertial/>
-		</link>
-		<gazebo reference="${prefix}thumb_prox">
-			<material>Gazebo/Grey</material>
-		</gazebo>
-		<!-- thumb med -->
-		<joint name="${prefix}thumb_med" type="fixed">
-			<origin xyz="0 0.00285 0.04341" rpy="0 0 0"/>
-			<parent link="${prefix}thumb_prox"/>
-			<child link="${prefix}thumb_med"/>
-		</joint>
-		<link name="${prefix}thumb_med">
-			<collision>
-				<origin xyz="0 0 0" rpy="0 0 0"/>
-				<geometry>
-					<mesh filename="package://hdt_7dof_description/meshes/thumb_med.stl"/>
-				</geometry>
-			</collision>
-			<visual>
-				<origin xyz="0 0 0" rpy="0 0 0"/>
-				<geometry>
-					<mesh filename="package://hdt_7dof_description/meshes/thumb_med.stl"/>
-				</geometry>
-				<material name="${prefix}black"/>
-			</visual>
-			<inertial>
-				<origin xyz="0 -0.00353 0.01162" rpy="0 0 0"/>
-				<mass value="0.0085"/>
-				<inertia
-					ixx="0.000001099" ixy="0.0" ixz="0.0"
-					iyy="0.000001639" iyz="0.000000096"
-					izz="0.000000981"/>
-			</inertial>
-		</link>
-		<gazebo reference="${prefix}thumb_med">
-			<material>Gazebo/Black</material>
-		</gazebo>
-		<!-- thumb dist -->
-		<joint name="${prefix}thumb_dist" type="fixed">
-			<origin xyz="0 -0.0009 0.02769" rpy="0 0 0"/>
-			<parent link="${prefix}thumb_med"/>
-			<child link="${prefix}thumb_dist"/>
-		</joint>
-		<link name="${prefix}thumb_dist">
-			<collision>
-				<origin xyz="0 0 0" rpy="0 0 0"/>
-				<geometry>
-					<mesh filename="package://hdt_7dof_description/meshes/thumb_dist.stl"/>
-				</geometry>
-			</collision>
-			<visual>
-				<origin xyz="0 0 0" rpy="0 0 0"/>
-				<geometry>
-					<mesh filename="package://hdt_7dof_description/meshes/thumb_dist.stl"/>
-				</geometry>
-				<material name="${prefix}grey"/>
-			</visual>
-			<inertial>
-				<origin xyz="0 -0.00131 0.01323" rpy="0 0 0"/>
-				<mass value="0.0092"/>
-				<inertia
-					ixx="0.00000066" ixy="0.0" ixz="0.0"
-					iyy="0.000000837" iyz="0.0"
-					izz="0.000000695"/>
-			</inertial>
-		</link>
-		<gazebo reference="${prefix}thumb_dist">
-			<material>Gazebo/Grey</material>
-		</gazebo>
-		<!-- index prox -->
-		<joint name="${prefix}index_yaw" type="revolute">
-			<hdt id="${motor_base_id + 11}" kmin="5" kmax="20" inertia="0.01"/>
-			<axis xyz="0 0 ${reflect*-1}"/>
-			<limit effort="4.0" lower="${left_only*-1.5708 + right_only*-0.7854}" upper="${left_only*0.7854 + right_only*1.5708}" velocity="4.1888"/>
-			<origin xyz="0 -0.16325 0.02701" rpy="0 ${left_only*3.1416} 0"/>
-			<parent link="${prefix}palm"/>
-			<child link="${prefix}index_prox"/>
-			<dynamics damping="0.7" friction="0.0"/>
-		</joint>
-		<transmission name="${prefix}tran12">
-			<type>transmission_interface/SimpleTransmission</type>
-			<joint name="${prefix}index_yaw">
-			</joint>
-			<actuator name="${prefix}motor12">
-				<hardwareInterface>EffortJointInterface</hardwareInterface>
-				<mechanicalReduction>1</mechanicalReduction>
-			</actuator>
-		</transmission>
-		<link name="${prefix}index_prox">
-			<collision>
-				<origin xyz="0 0 0" rpy="0 0 0"/>
-				<geometry>
-					<mesh filename="package://hdt_7dof_description/meshes/finger_prox_right.stl"/>
-				</geometry>
-			</collision>
-			<visual>
-				<origin xyz="0 0 0" rpy="0 0 0"/>
-				<geometry>
-					<mesh filename="package://hdt_7dof_description/meshes/finger_prox_right.stl"/>
-				</geometry>
-				<material name="${prefix}grey"/>
-			</visual>
-			<xacro:default_inertial/>
-		</link>
-		<gazebo reference="${prefix}index_prox">
-			<material>Gazebo/Grey</material>
-		</gazebo>
-		<!-- index med -->
-		<joint name="${prefix}index_med" type="fixed">
-			<origin xyz="-0.00285 -0.04341 0" rpy="0 0 0"/>
-			<parent link="${prefix}index_prox"/>
-			<child link="${prefix}index_med"/>
-		</joint>
-		<link name="${prefix}index_med">
-			<collision>
-				<origin xyz="0 0 0" rpy="0 0 0"/>
-				<geometry>
-					<mesh filename="package://hdt_7dof_description/meshes/finger_med_right.stl"/>
-				</geometry>
-			</collision>
-			<visual>
-				<origin xyz="0 0 0" rpy="0 0 0"/>
-				<geometry>
-					<mesh filename="package://hdt_7dof_description/meshes/finger_med_right.stl"/>
-				</geometry>
-				<material name="${prefix}black"/>
-			</visual>
-			<inertial>
-				<origin xyz="0.00353 -0.01162 0" rpy="0 0 0"/>
-				<mass value="0.0085"/>
-				<inertia
-					ixx="0.000001639" ixy="0.000000096" ixz="0.0"
-					iyy="0.000000981" iyz="0.0"
-					izz="0.000001099"/>
-			</inertial>
-		</link>
-		<gazebo reference="${prefix}index_med">
-			<material>Gazebo/Black</material>
-		</gazebo>
-		<!-- index dist -->
-		<joint name="${prefix}index_dist" type="fixed">
-			<origin xyz="0.0009 -0.02769 0" rpy="0 0 0"/>
-			<parent link="${prefix}index_med"/>
-			<child link="${prefix}index_dist"/>
-		</joint>
-		<link name="${prefix}index_dist">
-			<collision>
-				<origin xyz="0 0 0" rpy="0 0 0"/>
-				<geometry>
-					<mesh filename="package://hdt_7dof_description/meshes/finger_dist_right.stl"/>
-				</geometry>
-			</collision>
-			<visual>
-				<origin xyz="0 0 0" rpy="0 0 0"/>
-				<geometry>
-					<mesh filename="package://hdt_7dof_description/meshes/finger_dist_right.stl"/>
-				</geometry>
-				<material name="${prefix}grey"/>
-			</visual>
-			<inertial>
-				<origin xyz="0.00131 -0.01323 0" rpy="0 0 0"/>
-				<mass value="0.0092"/>
-				<inertia
-					ixx="0.000000837" ixy="0.0" ixz="0.0"
-					iyy="0.000000695" iyz="0.0"
-					izz="0.00000066"/>
-			</inertial>
-		</link>
-		<gazebo reference="${prefix}index_dist">
-			<material>Gazebo/Grey</material>
-		</gazebo>
-		<!-- ring prox -->
-		<joint name="${prefix}ring_yaw" type="revolute">
-			<hdt id="${motor_base_id + 12}" kmin="5" kmax="20" inertia="0.01"/>
-			<axis xyz="0 0 ${reflect*-1}"/>
-			<limit effort="4.0" lower="${left_only*-1.5708 + right_only*-0.7854}" upper="${left_only*0.7854 + right_only*1.5708}" velocity="4.1888"/>
-			<origin xyz="0 -0.16325 -0.02701" rpy="0 ${left_only*3.1416} 0"/>
-			<parent link="${prefix}palm"/>
-			<child link="${prefix}ring_prox"/>
-			<dynamics damping="0.7" friction="0.0"/>
-		</joint>
-		<transmission name="${prefix}tran13">
-			<type>transmission_interface/SimpleTransmission</type>
-			<joint name="${prefix}ring_yaw">
-			</joint>
-			<actuator name="${prefix}motor13">
-				<hardwareInterface>EffortJointInterface</hardwareInterface>
-				<mechanicalReduction>1</mechanicalReduction>
-			</actuator>
-		</transmission>
-		<link name="${prefix}ring_prox">
-			<collision>
-				<origin xyz="0 0 0" rpy="0 0 0"/>
-				<geometry>
-					<mesh filename="package://hdt_7dof_description/meshes/finger_prox_right.stl"/>
-				</geometry>
-			</collision>
-			<visual>
-				<origin xyz="0 0 0" rpy="0 0 0"/>
-				<geometry>
-					<mesh filename="package://hdt_7dof_description/meshes/finger_prox_right.stl"/>
-				</geometry>
-				<material name="${prefix}grey"/>
-			</visual>
-			<xacro:default_inertial/>
-		</link>
-		<gazebo reference="${prefix}ring_prox">
-			<material>Gazebo/Grey</material>
-		</gazebo>
-		<!-- ring med -->
-		<joint name="${prefix}ring_med" type="fixed">
-			<origin xyz="-0.00285 -0.04341 0" rpy="0 0 0"/>
-			<parent link="${prefix}ring_prox"/>
-			<child link="${prefix}ring_med"/>
-		</joint>
-		<link name="${prefix}ring_med">
-			<collision>
-				<origin xyz="0 0 0" rpy="0 0 0"/>
-				<geometry>
-					<mesh filename="package://hdt_7dof_description/meshes/finger_med_right.stl"/>
-				</geometry>
-			</collision>
-			<visual>
-				<origin xyz="0 0 0" rpy="0 0 0"/>
-				<geometry>
-					<mesh filename="package://hdt_7dof_description/meshes/finger_med_right.stl"/>
-				</geometry>
-				<material name="${prefix}black"/>
-			</visual>
-			<inertial>
-				<origin xyz="0.00353 -0.01162 0" rpy="0 0 0"/>
-				<mass value="0.0085"/>
-				<inertia
-					ixx="0.000001639" ixy="0.000000096" ixz="0.0"
-					iyy="0.000000981" iyz="0.0"
-					izz="0.000001099"/>
-			</inertial>
-		</link>
-		<gazebo reference="${prefix}ring_med">
-			<material>Gazebo/Black</material>
-		</gazebo>
-		<!-- ring dist -->
-		<joint name="${prefix}ring_dist" type="fixed">
-			<origin xyz="0.0009 -0.02769 0" rpy="0 0 0"/>
-			<parent link="${prefix}ring_med"/>
-			<child link="${prefix}ring_dist"/>
-		</joint>
-		<link name="${prefix}ring_dist">
-			<collision>
-				<origin xyz="0 0 0" rpy="0 0 0"/>
-				<geometry>
-					<mesh filename="package://hdt_7dof_description/meshes/finger_dist_right.stl"/>
-				</geometry>
-			</collision>
-			<visual>
-				<origin xyz="0 0 0" rpy="0 0 0"/>
-				<geometry>
-					<mesh filename="package://hdt_7dof_description/meshes/finger_dist_right.stl"/>
-				</geometry>
-				<material name="${prefix}grey"/>
-			</visual>
-			<inertial>
-				<origin xyz="0.00131 -0.01323 0" rpy="0 0 0"/>
-				<mass value="0.0092"/>
-				<inertia
-					ixx="0.000000837" ixy="0.0" ixz="0.0"
-					iyy="0.000000695" iyz="0.0"
-					izz="0.00000066"/>
-			</inertial>
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
Commit message: limited the elbow pitch upper limit

File: urdf/hdt_7dof_macro.xacro (robot description, xacro)
@@ -225,5 +225,5 @@
 			<hdt id="${motor_base_id + 3}" kmin="75" kmax="150" inertia="0.075"/>
 			<axis xyz="${reflect*-1} 0 0"/>
-			<limit effort="60.0" lower="-0.5236" upper="3.6652" velocity="2.0944"/>
+			<limit effort="60.0" lower="-0.5236" upper="2.0944" velocity="2.0944"/>
 			<origin xyz="0 0 -0.07" rpy="${left_only*3.1416} 0 0"/>
 			<parent link="${prefix}elbow_pitch_bracket"/>

File: urdf/hdt_7dof_macro_bbox.xacro (robot description, xacro)
@@ -171,5 +171,5 @@
 			<hdt id="${motor_base_id + 3}" kmin="75" kmax="150" inertia="0.075"/>
 			<axis xyz="${reflect*-1} 0 0"/>
-			<limit effort="60.0" lower="-0.5236" upper="3.6652" velocity="2.0944"/>
+			<limit effort="60.0" lower="-0.5236" upper="2.0944" velocity="2.0944"/>
 			<origin xyz="0 0 -0.07" rpy="${left_only*3.1416} 0 0"/>
 			<parent link="${prefix}elbow_pitch_bracket"/>

Commit message: limited the shoulder roll inward limits

File: urdf/hdt_7dof_macro.xacro (robot description, xacro)
@@ -104,5 +104,5 @@
 			<hdt id="${motor_base_id + 1}" kmin="100" kmax="200" inertia="0.1"/>
 			<axis xyz="0 ${reflect*1} 0"/>
-			<limit effort="60.0" lower="${left_only*-0.5236 + right_only*-3.1416}" upper="${left_only*3.1416 + right_only*0.5236}" velocity="2.0944"/>
+			<limit effort="60.0" lower="${left_only*-0.0 + right_only*-3.1416}" upper="${left_only*3.1416 + right_only*0.0}" velocity="2.0944"/>
 			<origin xyz="-0.07 0 0" rpy="0 0 0"/>
 			<parent link="${prefix}shoulder_roll_bracket"/>

File: urdf/hdt_7dof_macro_bbox.xacro (robot description, xacro)
@@ -85,5 +85,5 @@
 			<hdt id="${motor_base_id + 1}" kmin="100" kmax="200" inertia="0.1"/>
 			<axis xyz="0 ${reflect*1} 0"/>
-			<limit effort="60.0" lower="${left_only*-0.5236 + right_only*-3.1416}" upper="${left_only*3.1416 + right_only*0.5236}" velocity="2.0944"/>
+			<limit effort="60.0" lower="${left_only*-0.0 + right_only*-3.1416}" upper="${left_only*3.1416 + right_only*0.0}" velocity="2.0944"/>
 			<origin xyz="-0.07 0 0" rpy="0 0 0"/>
 			<parent link="${prefix}shoulder_roll_bracket"/>

Commit message: Add maroon as a colour for the mesh.

File: urdf/hdt_7dof_macro.xacro (robot description, xacro)
@@ -18,4 +18,7 @@
 			<color rgba="${53/255} ${94/255} ${59/255} 1.0"/>
 		</material>
+		<material name="${prefix}maroon">
+			<color rgba="${75/255} ${0/255} ${0/255} 1.0"/>
+		</material>
 		<material name="${prefix}black">
 			<color rgba="${0/255} ${0/255} ${0/255} 1.0"/>
@@ -55,5 +58,5 @@
 					<mesh filename="package://hdt_7dof_description/meshes/shoulder.stl"/>
 				</geometry>
-				<material name="${prefix}green"/>
+				<material name="${prefix}maroon"/>
 			</visual>
 			<inertial>
@@ -176,5 +179,5 @@
 					<mesh filename="package://hdt_7dof_description/meshes/upper_arm.stl"/>
 				</geometry>
-				<material name="${prefix}green"/>
+				<material name="${prefix}maroon"/>
 			</visual>
 			<inertial>
@@ -297,5 +300,5 @@
 					<mesh filename="package://hdt_7dof_description/meshes/forearm.stl"/>
 				</geometry>
-				<material name="${prefix}green"/>
+				<material name="${prefix}maroon"/>
 			</visual>
 			<inertial>

File: urdf/hdt_7dof_macro_bbox.xacro (robot description, xacro)
@@ -18,4 +18,7 @@
 			<color rgba="${53/255} ${94/255} ${59/255} 1.0"/>
 		</material>
+		<material name="${prefix}maroon">
+			<color rgba="${75/255} ${0/255} ${0/255} 1.0"/>
+		</material>
 		<material name="${prefix}black">
 			<color rgba="${0/255} ${0/255} ${0/255} 1.0"/>
@@ -70,5 +73,5 @@
 					<cylinder length="0.2" radius="0.05" />
 				</geometry>
-				<material name="${prefix}green"/>
+				<material name="${prefix}maroon"/>
 			</visual>
 			<inertial>
@@ -112,5 +115,5 @@
 					<cylinder length="0.32" radius="0.05"/>
 				</geometry>
-				<material name="${prefix}green"/>
+				<material name="${prefix}maroon"/>
 			</visual>
 			<inertial>
@@ -198,5 +201,5 @@
 					<cylinder length="0.1" radius="0.05"/>
 				</geometry>
-				<material name="${prefix}green"/>
+				<material name="${prefix}maroon"/>
 			</visual>
 			<inertial>
