Commit message: Add Gazebo material colors

File: urdf/hdt_7dof_left.xacro (robot description, xacro)
@@ -59,4 +59,7 @@
 		</inertial>
 	</link>
+	<gazebo reference="link1">
+		<material>Gazebo/Green</material>
+	</gazebo>
 	<joint name="joint1f" type="fixed">
 		<parent link="link1"/>
@@ -87,4 +90,7 @@
 		</inertial>
 	</link>
+	<gazebo reference="link2a">
+		<material>Gazebo/Black</material>
+	</gazebo>
 	<!-- segment 2 -->
 	<joint name="joint2" type="revolute">
@@ -129,4 +135,7 @@
 		</inertial>
 	</link>
+	<gazebo reference="link2b">
+		<material>Gazebo/Grey</material>
+	</gazebo>
 	<!-- segment 3 -->
 	<joint name="joint3" type="revolute">
@@ -162,4 +171,7 @@
 		</inertial>
 	</link>
+	<gazebo reference="link3">
+		<material>Gazebo/Green</material>
+	</gazebo>
 	<joint name="joint3f" type="fixed">
 		<origin xyz="0 0 -0.16271" rpy="0 0 0"/>
@@ -190,4 +202,7 @@
 		</inertial>
 	</link>
+	<gazebo reference="link4a">
+		<material>Gazebo/Black</material>
+	</gazebo>
 	<!-- segment 4 -->
 	<joint name="joint4" type="revolute">
@@ -232,4 +247,7 @@
 		</inertial>
 	</link>
+	<gazebo reference="link4b">
+		<material>Gazebo/Grey</material>
+	</gazebo>
 	<!-- segment 5 -->
 	<joint name="joint5" type="revolute">
@@ -274,4 +292,7 @@
 		</inertial>
 	</link>
+	<gazebo reference="link5">
+		<material>Gazebo/Green</material>
+	</gazebo>
 	<joint name="joint5f" type="fixed">
 		<origin xyz="0 -0.09217 0" rpy="0 0 0"/>
@@ -302,4 +323,7 @@
 		</inertial>
 	</link>
+	<gazebo reference="link6a">
+		<material>Gazebo/Black</material>
+	</gazebo>
 	<!-- segment 6 -->
 	<joint name="joint6" type="revolute">
@@ -344,4 +368,7 @@
 		</inertial>
 	</link>
+	<gazebo reference="link6b">
+		<material>Gazebo/Grey</material>
+	</gazebo>
 	<!-- segment 7 -->
 	<joint name="joint7" type="revolute">
@@ -386,4 +413,7 @@
 		</inertial>
 	</link>
+	<gazebo reference="link7">
+		<material>Gazebo/Black</material>
+	</gazebo>
 	<!-- palm -->
 	<joint name="palm" type="fixed">
@@ -415,4 +445,7 @@
 		</inertial>
 	</link>
+	<gazebo reference="palm">
+		<material>Gazebo/Black</material>
+	</gazebo>
 	<!-- thumb base -->
 	<joint name="thumb_base" type="revolute">
@@ -457,4 +490,7 @@
 		</inertial>
 	</link>
+	<gazebo reference="thumb_base">
+		<material>Gazebo/Grey</material>
+	</gazebo>
 	<!-- thumb prox -->
 	<joint name="thumb_prox" type="revolute">
@@ -499,4 +535,7 @@
 		</inertial>
 	</link>
+	<gazebo reference="thumb_prox">
+		<material>Gazebo/Grey</material>
+	</gazebo>
 	<!-- thumb med -->
 	<joint name="thumb_med" type="fixed">
@@ -528,4 +567,7 @@
 		</inertial>
 	</link>
+	<gazebo reference="thumb_med">
+		<material>Gazebo/Black</material>
+	</gazebo>
 	<!-- thumb dist -->
 	<joint name="thumb_dist" type="fixed">
@@ -557,4 +599,7 @@
 		</inertial>
 	</link>
+	<gazebo reference="thumb_dist">
+		<material>Gazebo/Grey</material>
+	</gazebo>
 	<!-- index prox -->
 	<joint name="index_prox" type="revolute">
@@ -599,4 +644,7 @@
 		</inertial>
 	</link>
+	<gazebo reference="index_prox">
+		<material>Gazebo/Grey</material>
+	</gazebo>
 	<!-- index med -->
 	<joint name="index_med" type="fixed">
@@ -628,4 +676,7 @@
 		</inertial>
 	</link>
+	<gazebo reference="index_med">
+		<material>Gazebo/Black</material>
+	</gazebo>
 	<!-- index dist -->
 	<joint name="index_dist" type="fixed">
@@ -657,4 +708,7 @@
 		</inertial>
 	</link>
+	<gazebo reference="index_dist">
+		<material>Gazebo/Grey</material>
+	</gazebo>
 	<!-- ring prox -->
 	<joint name="ring_prox" type="revolute">
@@ -699,4 +753,7 @@
 		</inertial>
 	</link>
+	<gazebo reference="ring_prox">
+		<material>Gazebo/Grey</material>
+	</gazebo>
 	<!-- ring med -->
 	<joint name="ring_med" type="fixed">
@@ -728,4 +785,7 @@
 		</inertial>
 	</link>
+	<gazebo reference="ring_med">
+		<material>Gazebo/Black</material>
+	</gazebo>
 	<!-- ring dist -->
 	<joint name="ring_dist" type="fixed">
@@ -757,3 +817,6 @@
 		</inertial>
 	</link>
+	<gazebo reference="ring_dist">
+		<material>Gazebo/Grey</material>
+	</gazebo>
 </robot>

File: urdf/hdt_7dof_right.xacro (robot description, xacro)
@@ -59,4 +59,7 @@
 		</inertial>
 	</link>
+	<gazebo reference="link1">
+		<material>Gazebo/Green</material>
+	</gazebo>
 	<joint name="joint1f" type="fixed">
 		<parent link="link1"/>
@@ -87,4 +90,7 @@
 		</inertial>
 	</link>
+	<gazebo reference="link2a">
+		<material>Gazebo/Black</material>
+	</gazebo>
 	<!-- segment 2 -->
 	<joint name="joint2" type="revolute">
@@ -129,4 +135,7 @@
 		</inertial>
 	</link>
+	<gazebo reference="link2b">
+		<material>Gazebo/Grey</material>
+	</gazebo>
 	<!-- segment 3 -->
 	<joint name="joint3" type="revolute">
@@ -162,4 +171,7 @@
 		</inertial>
 	</link>
+	<gazebo reference="link3">
+		<material>Gazebo/Green</material>
+	</gazebo>
 	<joint name="joint3f" type="fixed">
 		<origin xyz="0 0 -0.16271" rpy="0 0 0"/>
@@ -190,4 +202,7 @@
 		</inertial>
 	</link>
+	<gazebo reference="link4a">
+		<material>Gazebo/Black</material>
+	</gazebo>
 	<!-- segment 4 -->
 	<joint name="joint4" type="revolute">
@@ -232,4 +247,7 @@
 		</inertial>
 	</link>
+	<gazebo reference="link4b">
+		<material>Gazebo/Grey</material>
+	</gazebo>
 	<!-- segment 5 -->
 	<joint name="joint5" type="revolute">
@@ -274,4 +292,7 @@
 		</inertial>
 	</link>
+	<gazebo reference="link5">
+		<material>Gazebo/Green</material>
+	</gazebo>
 	<joint name="joint5f" type="fixed">
 		<origin xyz="0 -0.09217 0" rpy="0 0 0"/>
@@ -302,4 +323,7 @@
 		</inertial>
 	</link>
+	<gazebo reference="link6a">
+		<material>Gazebo/Black</material>
+	</gazebo>
 	<!-- segment 6 -->
 	<joint name="joint6" type="revolute">
@@ -344,4 +368,7 @@
 		</inertial>
 	</link>
+	<gazebo reference="link6b">
+		<material>Gazebo/Grey</material>
+	</gazebo>
 	<!-- segment 7 -->
 	<joint name="joint7" type="revolute">
@@ -386,4 +413,7 @@
 		</inertial>
 	</link>
+	<gazebo reference="link7">
+		<material>Gazebo/Black</material>
+	</gazebo>
 	<!-- palm -->
 	<joint name="palm" type="fixed">
@@ -415,4 +445,7 @@
 		</inertial>
 	</link>
+	<gazebo reference="palm">
+		<material>Gazebo/Black</material>
+	</gazebo>
 	<!-- thumb base -->
 	<joint name="thumb_base" type="revolute">
@@ -457,4 +490,7 @@
 		</inertial>
 	</link>
+	<gazebo reference="thumb_base">
+		<material>Gazebo/Grey</material>
+	</gazebo>
 	<!-- thumb prox -->
 	<joint name="thumb_prox" type="revolute">
@@ -499,4 +535,7 @@
 		</inertial>
 	</link>
+	<gazebo reference="thumb_prox">
+		<material>Gazebo/Grey</material>
+	</gazebo>
 	<!-- thumb med -->
 	<joint name="thumb_med" type="fixed">
@@ -528,4 +567,7 @@
 		</inertial>
 	</link>
+	<gazebo reference="thumb_med">
+		<material>Gazebo/Black</material>
+	</gazebo>
 	<!-- thumb dist -->
 	<joint name="thumb_dist" type="fixed">
@@ -557,4 +599,7 @@
 		</inertial>
 	</link>
+	<gazebo reference="thumb_dist">
+		<material>Gazebo/Grey</material>
+	</gazebo>
 	<!-- index prox -->
 	<joint name="index_prox" type="revolute">
@@ -599,4 +644,7 @@
 		</inertial>
 	</link>
+	<gazebo reference="index_prox">
+		<material>Gazebo/Grey</material>
+	</gazebo>
 	<!-- index med -->
 	<joint name="index_med" type="fixed">
@@ -628,4 +676,7 @@
 		</inertial>
 	</link>
+	<gazebo reference="index_med">
+		<material>Gazebo/Black</material>
+	</gazebo>
 	<!-- index dist -->
 	<joint name="index_dist" type="fixed">
@@ -657,4 +708,7 @@
 		</inertial>
 	</link>
+	<gazebo reference="index_dist">
+		<material>Gazebo/Grey</material>
+	</gazebo>
 	<!-- ring prox -->
 	<joint name="ring_prox" type="revolute">
@@ -699,4 +753,7 @@
 		</inertial>
 	</link>
+	<gazebo reference="ring_prox">
+		<material>Gazebo/Grey</material>
+	</gazebo>
 	<!-- ring med -->
 	<joint name="ring_med" type="fixed">
@@ -728,4 +785,7 @@
 		</inertial>
 	</link>
+	<gazebo reference="ring_med">
+		<material>Gazebo/Black</material>
+	</gazebo>
 	<!-- ring dist -->
 	<joint name="ring_dist" type="fixed">
@@ -757,3 +817,6 @@
 		</inertial>
 	</link>
+	<gazebo reference="ring_dist">
+		<material>Gazebo/Grey</material>
+	</gazebo>
 </robot>

Commit message: Rename base_link to world
"world" is a special link name for Gazebo, and means that the link
will be treated as fixed.

File: urdf/hdt_7dof_left.xacro (robot description, xacro)
@@ -23,5 +23,5 @@
 	<xacro:include filename="$(find hdt_7dof_description)/urdf/hdt_7dof.gazebo" /> -->
 	<!-- segment 0 -->
-	<link name="base_link"/>
+	<link name="world" />
 	<!-- segment 1 -->
 	<joint name="joint1" type="revolute">
@@ -30,5 +30,5 @@
 		<limit effort="60.0" lower="-3.1416" upper="1.0472" velocity="2.0944"/>
 		<origin xyz="0 0 0" rpy="0 0 3.1416"/>
-		<parent link="base_link"/>
+		<parent link="world"/>
 		<child link="link1"/>
     		<dynamics damping="0.7" friction="0.0"/>

File: urdf/hdt_7dof_right.xacro (robot description, xacro)
@@ -23,5 +23,5 @@
 	<xacro:include filename="$(find hdt_7dof_description)/urdf/hdt_7dof.gazebo" /> -->
 	<!-- segment 0 -->
-	<link name="base_link"/>
+	<link name="world" />
 	<!-- segment 1 -->
 	<joint name="joint1" type="revolute">
@@ -30,5 +30,5 @@
 		<limit effort="60.0" lower="-3.1416" upper="1.0472" velocity="2.0944"/>
 		<origin xyz="0 0 0" rpy="0 0 0"/>
-		<parent link="base_link"/>
+		<parent link="world"/>
 		<child link="link1"/>
     		<dynamics damping="0.7" friction="0.0"/>

Commit message: Increase inertia of _prox links
This allows Gazebo to correctly simulate the arms even
with the joint limits.

File: urdf/hdt_7dof_left.xacro (robot description, xacro)
@@ -3,4 +3,11 @@
 	<!-- constants -->
 	<xacro:property name="PI" value="3.1415926535897931"/>
+	<!-- default inertia -->
+	<xacro:macro name="default_inertia">
+		<inertia
+		ixx="0.0005" ixy="0.0" ixz="0.0"
+		iyy="0.0005" iyz="0.0"
+		izz="0.0005"/>
+	</xacro:macro>
 	<!-- materials -->
 	<material name="green">
@@ -529,8 +536,9 @@
 			<origin xyz="0 0.001 0.02063" rpy="0 0 0"/>
 			<mass value="0.02523"/>
-			<inertia
+			<xacro:default_inertia />
+			<!-- <inertia
 			ixx="0.000004718" ixy="0.0" ixz="0.0"
 			iyy="0.000005374" iyz="-0.000000071"
-			izz="0.000002921"/>
+			izz="0.000002921"/> -->
 		</inertial>
 	</link>
@@ -638,8 +646,9 @@
 			<origin xyz="-0.001 -0.02063 0" rpy="0 0 0"/>
 			<mass value="0.02523"/>
-			<inertia
+			<xacro:default_inertia />
+			<!-- <inertia
 			ixx="0.000005374" ixy="-0.000000071" ixz="0.0"
 			iyy="0.000002921" iyz="0.0"
-			izz="0.000004718"/>
+			izz="0.000004718"/> -->
 		</inertial>
 	</link>
@@ -747,8 +756,9 @@
 			<origin xyz="-0.001 -0.02063 0" rpy="0 0 0"/>
 			<mass value="0.02523"/>
-			<inertia
+			<xacro:default_inertia />
+			<!-- <inertia
 			ixx="0.000005374" ixy="-0.000000071" ixz="0.0"
 			iyy="0.000002921" iyz="0.0"
-			izz="0.000004718"/>
+			izz="0.000004718"/> -->
 		</inertial>
 	</link>

File: urdf/hdt_7dof_right.xacro (robot description, xacro)
@@ -3,4 +3,11 @@
 	<!-- constants -->
 	<xacro:property name="PI" value="3.1415926535897931"/>
+	<!-- default inertia -->
+	<xacro:macro name="default_inertia">
+		<inertia
+		ixx="0.0005" ixy="0.0" ixz="0.0"
+		iyy="0.0005" iyz="0.0"
+		izz="0.0005"/>
+	</xacro:macro>
 	<!-- materials -->
 	<material name="green">
@@ -529,8 +536,9 @@
 			<origin xyz="0 0.001 0.02063" rpy="0 0 0"/>
 			<mass value="0.02523"/>
-			<inertia
+			<xacro:default_inertia />
+			<!-- <inertia
 			ixx="0.000004718" ixy="0.0" ixz="0.0"
 			iyy="0.000005374" iyz="-0.000000071"
-			izz="0.000002921"/>
+			izz="0.000002921"/> -->
 		</inertial>
 	</link>
@@ -638,8 +646,9 @@
 			<origin xyz="-0.001 -0.02063 0" rpy="0 0 0"/>
 			<mass value="0.02523"/>
-			<inertia
+			<xacro:default_inertia />
+			<!-- <inertia
 			ixx="0.000005374" ixy="-0.000000071" ixz="0.0"
 			iyy="0.000002921" iyz="0.0"
-			izz="0.000004718"/>
+			izz="0.000004718"/> -->
 		</inertial>
 	</link>
@@ -747,8 +756,9 @@
 			<origin xyz="-0.001 -0.02063 0" rpy="0 0 0"/>
 			<mass value="0.02523"/>
-			<inertia
+			<xacro:default_inertia />
+			<!-- <inertia
 			ixx="0.000005374" ixy="-0.000000071" ixz="0.0"
 			iyy="0.000002921" iyz="0.0"
-			izz="0.000004718"/>
+			izz="0.000004718"/> -->
 		</inertial>
 	</link>

Commit message: Add transmission for joint3

File: urdf/hdt_7dof_left.xacro (robot description, xacro)
@@ -155,4 +155,13 @@
     		<dynamics damping="0.7" friction="0.0"/>
 	</joint>
+	<transmission name="tran3">
+		<type>transmission_interface/SimpleTransmission</type>
+		<joint name="joint3">
+			<hardwareInterface>EffortJointInterface</hardwareInterface>
+		</joint>
+		<actuator name="motor3">
+			<mechanicalReduction>1</mechanicalReduction>
+		</actuator>
+	</transmission>
 	<link name="link3">
 		<collision>

File: urdf/hdt_7dof_right.xacro (robot description, xacro)
@@ -155,4 +155,13 @@
     		<dynamics damping="0.7" friction="0.0"/>
 	</joint>
+	<transmission name="tran3">
+		<type>transmission_interface/SimpleTransmission</type>
+		<joint name="joint3">
+			<hardwareInterface>EffortJointInterface</hardwareInterface>
+		</joint>
+		<actuator name="motor3">
+			<mechanicalReduction>1</mechanicalReduction>
+		</actuator>
+	</transmission>
 	<link name="link3">
 		<collision>
