Commit message: Break out arms into macro files
This allows them to be reused wholesale in robots.

File: urdf/hdt_7dof_right.xacro (robot description, xacro)
@@ -6,841 +6,7 @@
 		</plugin>
 	</gazebo>
-	<!-- constants -->
-	<xacro:property name="PI" value="3.1415926535897931"/>
-	<!-- default inertia -->
-	<xacro:macro name="default_inertia">
-		<inertia
-		ixx="0.0005" ixy="0.0" ixz="0.0"
-		iyy="0.0005" iyz="0.0"
-		izz="0.0005"/>
-	</xacro:macro>
-	<!-- materials -->
-	<material name="green">
-		<color rgba="${53/255} ${94/255} ${59/255} 1.0"/>
-	</material>
-	<material name="black">
-		<color rgba="${0/255} ${0/255} ${0/255} 1.0"/>
-	</material>
-	<material name="grey">
-		<color rgba="${40/255} ${40/255} ${40/255} 1.0"/>
-	</material>
-	<!-- import gazebo definitions
-	<xacro:include filename="$(find hdt_7dof_description)/urdf/hdt_7dof.gazebo" /> -->
 	<!-- segment 0 -->
 	<link name="world" />
-	<!-- segment 1 -->
-	<joint name="joint1" type="revolute">
-		<hdt id="1" kmin="100" kmax="200" inertia="0.1"/>
-		<axis xyz="1 0 0"/>
-		<limit effort="60.0" lower="-3.1416" upper="1.0472" velocity="2.0944"/>
-		<origin xyz="0 0 0" rpy="0 0 0"/>
-		<parent link="world"/>
-		<child link="link1"/>
-    		<dynamics damping="0.7" friction="0.0"/>
-	</joint>
-	<transmission name="tran1">
-		<type>transmission_interface/SimpleTransmission</type>
-		<joint name="joint1">
-			<hardwareInterface>EffortJointInterface</hardwareInterface>
-		</joint>
-		<actuator name="motor1">
-			<mechanicalReduction>1</mechanicalReduction>
-		</actuator>
-	</transmission>
-	<link name="link1">
-		<collision>
-			<origin xyz="0 0 0" rpy="0 0 0"/>
-			<geometry>
-				<mesh filename="package://hdt_7dof_description/meshes/hdt_7dof_1_right.STL"/>
-			</geometry>
-		</collision>
-		<visual>
-			<origin xyz="0 0 0" rpy="0 0 0"/>
-			<geometry>
-				<mesh filename="package://hdt_7dof_description/meshes/hdt_7dof_1_right.STL"/>
-			</geometry>
-			<material name="green"/>
-		</visual>
-		<inertial>
-		<origin xyz="-0.04488 0 0" rpy="0 0 0"/>
-		<mass value="1.00775"/>
-			<inertia
-			ixx="0.00064952" ixy="0.0" ixz="0.0"
-			iyy="0.00104342" iyz="0.0"
-			izz="0.00104342"/>
-		</inertial>
-	</link>
-	<gazebo reference="link1">
-		<material>Gazebo/Green</material>
-	</gazebo>
-	<joint name="joint1f" type="fixed">
-		<parent link="link1"/>
-		<child link="link2a"/>
-		<origin xyz="-0.09217 0 0" rpy="0 0 0"/>
-	</joint>
-	<link name="link2a">
-		<collision>
-			<origin xyz="0 0 0" rpy="0 0 0"/>
-			<geometry>
-				<mesh filename="package://hdt_7dof_description/meshes/hdt_7dof_2a_right.STL"/>
-			</geometry>
-		</collision>
-		<visual>
-			<origin xyz="0 0 0" rpy="0 0 0"/>
-			<geometry>
-				<mesh filename="package://hdt_7dof_description/meshes/hdt_7dof_2a_right.STL"/>
-			</geometry>
-			<material name="black"/>
-		</visual>
-		<inertial>
-			<origin xyz="-0.04416876 0 0" rpy="0 0 0"/>
-			<mass value="0.66774822"/>
-			<inertia
-			ixx="0.00062987" ixy="0.0" ixz="0.0"
-			iyy="0.00091291" iyz="0.0"
-			izz="0.00110241"/>
-		</inertial>
-	</link>
-	<gazebo reference="link2a">
-		<material>Gazebo/Black</material>
-	</gazebo>
-	<!-- segment 2 -->
-	<joint name="joint2" type="revolute">
-		<hdt id="2" kmin="100" kmax="200" inertia="0.1"/>
-		<axis xyz="0 -1 0"/>
-		<limit effort="60.0" lower="-3.1416" upper="0.5236" velocity="2.0944"/>
-		<origin xyz="-0.07 0 0" rpy="0 0 0"/>
-		<parent link="link2a"/>
-		<child link="link2b"/>
-    		<dynamics damping="0.7" friction="0.0"/>
-	</joint>
-	<transmission name="tran2">
-		<type>transmission_interface/SimpleTransmission</type>
-		<joint name="joint2">
-			<hardwareInterface>EffortJointInterface</hardwareInterface>
-		</joint>
-		<actuator name="motor2">
-			<mechanicalReduction>1</mechanicalReduction>
-		</actuator>
-	</transmission>
-	<link name="link2b">
-		<collision>
-			<origin xyz="0 0 0" rpy="0 0 0"/>
-			<geometry>
-				<mesh filename="package://hdt_7dof_description/meshes/hdt_7dof_2b.STL"/>
-			</geometry>
-		</collision>
-		<visual>
-			<origin xyz="0 0 0.0" rpy="0 0 0"/>
-			<geometry>
-				<mesh filename="package://hdt_7dof_description/meshes/hdt_7dof_2b.STL"/>
-			</geometry>
-			<material name="grey"/>
-		</visual>
-		<inertial>
-			<origin xyz="0 0 -0.02018105" rpy="0 0 0"/>
-			<mass value="0.69896"/>
-			<inertia
-			ixx="0.00088116" ixy="0.0" ixz="0.0"
-			iyy="0.00094182" iyz="0.0"
-			izz="0.00032992"/>
-		</inertial>
-	</link>
-	<gazebo reference="link2b">
-		<material>Gazebo/Grey</material>
-	</gazebo>
-	<!-- segment 3 -->
-	<joint name="joint3" type="revolute">
-		<hdt id="3" kmin="75" kmax="150" inertia="0.075"/>
-		<axis xyz="0 0 1"/>
-		<limit effort="60.0" lower="-2.0944" upper="2.0944" velocity="2.0944"/>
-		<origin xyz="0 0 -0.077" rpy="0 0 0" />
-		<parent link="link2b"/>
-		<child link="link3"/>
-    		<dynamics damping="0.7" friction="0.0"/>
-	</joint>
-	<transmission name="tran3">
-		<type>transmission_interface/SimpleTransmission</type>
-		<joint name="joint3">
-			<hardwareInterface>EffortJointInterface</hardwareInterface>
-		</joint>
-		<actuator name="motor3">
-			<mechanicalReduction>1</mechanicalReduction>
-		</actuator>
-	</transmission>
-	<link name="link3">
-		<collision>
-			<origin xyz="0 0 0.0" rpy="0 0 0"/>
-			<geometry>
-				<mesh filename="package://hdt_7dof_description/meshes/hdt_7dof_3.STL"/>
-			</geometry>
-		</collision>
-		<visual>
-			<origin xyz="0 0 0.0" rpy="0 0 0"/>
-			<geometry>
-				<mesh filename="package://hdt_7dof_description/meshes/hdt_7dof_3.STL"/>
-			</geometry>
-			<material name="green"/>
-		</visual>
-		<inertial>
-			<origin xyz="0 0 -0.08013953" rpy="0 0 0"/>
-			<mass value="1.77733729"/>
-			<inertia
-			ixx="0.00450640" ixy="0.0" ixz="0.0"
-			iyy="0.00450640" iyz="0.0"
-			izz="0.00114447"/>
-		</inertial>
-	</link>
-	<gazebo reference="link3">
-		<material>Gazebo/Green</material>
-	</gazebo>
-	<joint name="joint3f" type="fixed">
-		<origin xyz="0 0 -0.16271" rpy="0 0 0"/>
-		<parent link="link3"/>
-		<child link="link4a"/>
-	</joint>
-	<link name="link4a">
-		<collision>
-			<origin xyz="0 0 0" rpy="0 0 0"/>
-			<geometry>
-				<mesh filename="package://hdt_7dof_description/meshes/hdt_7dof_4a.STL"/>
-			</geometry>
-		</collision>
-		<visual>
-			<origin xyz="0 0 0.0" rpy="0 0 0"/>
-			<geometry>
-				<mesh filename="package://hdt_7dof_description/meshes/hdt_7dof_4a.STL"/>
-			</geometry>
-			<material name="black"/>
-		</visual>
-		<inertial>
-			<origin xyz="0 0 -0.04416876" rpy="0 0 0"/>
-			<mass value="0.66774822"/>
-			<inertia
-			ixx="0.00091291" ixy="0.0" ixz="0.0"
-			iyy="0.00110241" iyz="0.0"
-			izz="0.00062987"/>
-		</inertial>
-	</link>
-	<gazebo reference="link4a">
-		<material>Gazebo/Black</material>
-	</gazebo>
-	<!-- segment 4 -->
-	<joint name="joint4" type="revolute">
-		<hdt id="4" kmin="75" kmax="150" inertia="0.075"/>
-		<axis xyz="1 0 0"/>
-		<limit effort="60.0" lower="-0.5236" upper="3.6652" velocity="2.0944"/>
-		<origin xyz="0 0 -0.07" rpy="0 0 0"/>
-		<parent link="link4a"/>
-		<child link="link4b"/>
-		<dynamics damping="0.7" friction="0.0"/>
-	</joint>
-	<transmission name="tran4">
-		<type>transmission_interface/SimpleTransmission</type>
-		<joint name="joint4">
-			<hardwareInterface>EffortJointInterface</hardwareInterface>
-		</joint>
-		<actuator name="motor4">
-			<mechanicalReduction>1</mechanicalReduction>
-		</actuator>
-	</transmission>
-	<link name="link4b">
-		<collision>
-			<origin xyz="0 0 0" rpy="0 0 0"/>
-			<geometry>
-				<mesh filename="package://hdt_7dof_description/meshes/hdt_7dof_4b.STL"/>
-			</geometry>
-		</collision>
-		<visual>
-			<origin xyz="0 0 0.0" rpy="0 0 0"/>
-			<geometry>
-				<mesh filename="package://hdt_7dof_description/meshes/hdt_7dof_4b.STL"/>
-			</geometry>
-			<material name="grey"/>
-		</visual>
-		<inertial>
-			<origin xyz="0 -0.02018105 0" rpy="0 0 0"/>
-			<mass value="0.69896279"/>
-			<inertia
-			ixx="0.00094182" ixy="0.0" ixz="0.0"
-			iyy="0.00032992" iyz="0.0"
-			izz="0.00088116"/>
-		</inertial>
-	</link>
-	<gazebo reference="link4b">
-		<material>Gazebo/Grey</material>
-	</gazebo>
-	<!-- segment 5 -->
-	<joint name="joint5" type="revolute">
-		<hdt id="5" kmin="50" kmax="100" inertia="0.05"/>
-		<axis xyz="0 -1 0"/>
-		<limit effort="60.0" lower="-2.0944" upper="2.0944" velocity="2.0944"/>
-		<origin xyz="0 -0.077 0" rpy="0 0 0"/>
-		<parent link="link4b"/>
-		<child link="link5"/>
-		<dynamics damping="0.7" friction="0.0"/>
-	</joint>
-	<transmission name="tran5">
-		<type>transmission_interface/SimpleTransmission</type>
-		<joint name="joint5">
-			<hardwareInterface>EffortJointInterface</hardwareInterface>
-		</joint>
-		<actuator name="motor5">
-			<mechanicalReduction>1</mechanicalReduction>
-		</actuator>
-	</transmission>
-	<link name="link5">
-		<collision>
-			<origin xyz="0 0 0.0" rpy="0 0 0"/>
-			<geometry>
-				<mesh filename="package://hdt_7dof_description/meshes/hdt_7dof_5.STL"/>
-			</geometry>
-		</collision>
-		<visual>
-			<origin xyz="0 0 0.0" rpy="0 0 0"/>
-			<geometry>
-				<mesh filename="package://hdt_7dof_description/meshes/hdt_7dof_5.STL"/>
-			</geometry>
-			<material name="green"/>
-		</visual>
-		<inertial>
-			<origin xyz="0 -0.04487724 0" rpy="0 0 0"/>
-			<mass value="1.00775488"/>
-			<inertia
-			ixx="0.00104342" ixy="0.0" ixz="0.0"
-			iyy="0.00064952" iyz="0.0"
-			izz="0.00104342"/>
-		</inertial>
-	</link>
-	<gazebo reference="link5">
-		<material>Gazebo/Green</material>
-	</gazebo>
-	<joint name="joint5f" type="fixed">
-		<origin xyz="0 -0.09217 0" rpy="0 0 0"/>
-		<parent link="link5"/>
-		<child link="link6a"/>
-	</joint>
-	<link name="link6a">
-		<collision>
-			<origin xyz="0 0 0" rpy="0 0 0"/>
-			<geometry>
-				<mesh filename="package://hdt_7dof_description/meshes/hdt_7dof_6a.STL"/>
-			</geometry>
-		</collision>
-		<visual>
-			<origin xyz="0 0 0.0" rpy="0 0 0"/>
-			<geometry>
-				<mesh filename="package://hdt_7dof_description/meshes/hdt_7dof_6a.STL"/>
-			</geometry>
-			<material name="black"/>
-		</visual>
-		<inertial>
-			<origin xyz="0 -0.04112 0" rpy="0 0 0"/>
-			<mass value="0.50058"/>
-			<inertia
-			ixx="0.000580228" ixy="0.0" ixz="0.0"
-			iyy="0.000541503" iyz="0.0"
-			izz="0.000750977"/>
-		</inertial>
-	</link>
-	<gazebo reference="link6a">
-		<material>Gazebo/Black</material>
-	</gazebo>
-	<!-- segment 6 -->
-	<joint name="joint6" type="revolute">
-		<hdt id="6" kmin="50" kmax="100" inertia="0.05"/>
-		<axis xyz="1 0 0"/>
-		<limit effort="60.0" lower="-1.5708" upper="1.5708" velocity="2.0944"/>
-		<origin xyz="0 -0.055 0" rpy="0 0 0"/>
-		<parent link="link6a"/>
-		<child link="link6b"/>
-		<dynamics damping="0.7" friction="0.0"/>
-	</joint>
-	<transmission name="tran6">
-		<type>transmission_interface/SimpleTransmission</type>
-		<joint name="joint6">
-			<hardwareInterface>EffortJointInterface</hardwareInterface>
-		</joint>
-		<actuator name="motor6">
-			<mechanicalReduction>1</mechanicalReduction>
-		</actuator>
-	</transmission>
-	<link name="link6b">
-		<collision>
-			<origin xyz="0 0 0" rpy="0 0 0"/>
-			<geometry>
-				<mesh filename="package://hdt_7dof_description/meshes/hdt_7dof_6b.STL"/>
-			</geometry>
-		</collision>
-		<visual>
-			<origin xyz="0 0 0.0" rpy="0 0 0"/>
-			<geometry>
-				<mesh filename="package://hdt_7dof_description/meshes/hdt_7dof_6b.STL"/>
-			</geometry>
-			<material name="grey"/>
-		</visual>
-		<inertial>
-			<origin xyz="0 -0.03855 0" rpy="0 0 0"/>
-			<mass value="0.99934"/>
-			<inertia
-			ixx="0.001905243" ixy="0.0" ixz="0.0"
-			iyy="0.000474765" iyz="0.0"
-			izz="0.001905243"/>
-		</inertial>
-	</link>
-	<gazebo reference="link6b">
-		<material>Gazebo/Grey</material>
-	</gazebo>
-	<!-- segment 7 -->
-	<joint name="joint7" type="revolute">
-		<hdt id="7" kmin="50" kmax="100" inertia="0.05"/>
-		<axis xyz="0 0 1"/>
-		<limit effort="60.0" lower="-1.5708" upper="1.5708" velocity="2.0944"/>
-		<origin xyz="0 -0.0771 0" rpy="0 0 0"/>
-		<parent link="link6b"/>
-		<child link="link7"/>
-		<dynamics damping="0.7" friction="0.0"/>
-	</joint>
-	<transmission name="tran7">
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
Commit message: Arm macro takes a yaw argument

File: urdf/hdt_7dof_left.xacro (robot description, xacro)
@@ -9,4 +9,4 @@
 	<link name="world" />
 	<xacro:include filename="$(find hdt_7dof_description)/urdf/hdt_7dof_left_macro.xacro" />
-	<xacro:hdt_7dof_left parent="world" x="0" y="0" z="0" />
+	<xacro:hdt_7dof_left parent="world" x="0" y="0" z="0" yaw="-1.57079" />
 </robot>

File: urdf/hdt_7dof_left_macro.xacro (robot description, xacro)
@@ -8,5 +8,5 @@
 		izz="0.0005"/>
 	</xacro:macro>
-	<xacro:macro name="hdt_7dof_left" params="parent x y z">
+	<xacro:macro name="hdt_7dof_left" params="parent x y z yaw">
 		<!-- materials -->
 		<material name="green">
@@ -24,5 +24,5 @@
 			<axis xyz="-1 0 0"/>
 			<limit effort="60.0" lower="-3.1416" upper="1.0472" velocity="2.0944"/>
-			<origin xyz="${x} ${y} ${z}" rpy="0 0 3.1416"/>
+			<origin xyz="${x} ${y} ${z}" rpy="0 0 ${yaw}"/>
 			<parent link="${parent}"/>
 			<child link="link1"/>

File: urdf/hdt_7dof_right.xacro (robot description, xacro)
@@ -9,4 +9,4 @@
 	<link name="world" />
 	<xacro:include filename="$(find hdt_7dof_description)/urdf/hdt_7dof_right_macro.xacro" />
-	<xacro:hdt_7dof_right parent="world" x="0" y="0" z="0" />
+	<xacro:hdt_7dof_right parent="world" x="0" y="0" z="0" yaw="1.57079" />
 </robot>

File: urdf/hdt_7dof_right_macro.xacro (robot description, xacro)
@@ -8,5 +8,5 @@
 		izz="0.0005"/>
 	</xacro:macro>
-	<xacro:macro name="hdt_7dof_right" params="parent x y z">
+	<xacro:macro name="hdt_7dof_right" params="parent x y z yaw">
 		<!-- materials -->
 		<material name="green">
@@ -24,5 +24,5 @@
 			<axis xyz="1 0 0"/>
 			<limit effort="60.0" lower="-3.1416" upper="1.0472" velocity="2.0944"/>
-			<origin xyz="${x} ${y} ${z}" rpy="0 0 0"/>
+			<origin xyz="${x} ${y} ${z}" rpy="0 0 ${yaw}"/>
 			<parent link="${parent}"/>
 			<child link="link1"/>
