Commit message: changed to allow an input yaw orientation and prefix

File: urdf/hdt_7dof_left.xacro (robot description, xacro)
@@ -9,4 +9,4 @@
 	<link name="world" />
 	<xacro:include filename="$(find hdt_7dof_description)/urdf/hdt_7dof_left_macro.xacro" />
-	<xacro:hdt_7dof_left parent="world" x="0" y="0" z="0" />
+	<xacro:hdt_7dof_left parent="world" x="0" y="0" z="0" yaw="3.1416" prefix="" />
 </robot>

File: urdf/hdt_7dof_left_macro.xacro (robot description, xacro)
@@ -8,35 +8,35 @@
 		izz="0.0005"/>
 	</xacro:macro>
-	<xacro:macro name="hdt_7dof_left" params="parent x y z">
+	<xacro:macro name="hdt_7dof_left" params="parent x y z yaw prefix">
 		<!-- materials -->
-		<material name="green">
+		<material name="${prefix}green">
 			<color rgba="${53/255} ${94/255} ${59/255} 1.0"/>
 		</material>
-		<material name="black">
+		<material name="${prefix}black">
 			<color rgba="${0/255} ${0/255} ${0/255} 1.0"/>
 		</material>
-		<material name="grey">
+		<material name="${prefix}grey">
 			<color rgba="${40/255} ${40/255} ${40/255} 1.0"/>
 		</material>
 		<!-- segment 1 -->
-		<joint name="joint1" type="revolute">
+		<joint name="${prefix}joint1" type="revolute">
 			<hdt id="41" kmin="100" kmax="200" inertia="0.1"/>
 			<axis xyz="-1 0 0"/>
 			<limit effort="60.0" lower="-3.1416" upper="1.0472" velocity="2.0944"/>
-			<origin xyz="${x} ${y} ${z}" rpy="0 0 3.1416"/>
+			<origin xyz="${x} ${y} ${z}" rpy="0 0 ${yaw}"/>
 			<parent link="${parent}"/>
-			<child link="link1"/>
-			<dynamics damping="0.7" friction="0.0"/>
-		</joint>
-		<transmission name="tran1">
-			<type>transmission_interface/SimpleTransmission</type>
-			<joint name="joint1">
-				<hardwareInterface>EffortJointInterface</hardwareInterface>
-			</joint>
-			<actuator name="motor1">
-				<mechanicalReduction>1</mechanicalReduction>
-			</actuator>
-		</transmission>
-		<link name="link1">
+			<child link="${prefix}link1"/>
+			<dynamics damping="0.7" friction="0.0"/>
+		</joint>
+		<transmission name="${prefix}tran1">
+			<type>transmission_interface/SimpleTransmission</type>
+			<joint name="${prefix}joint1">
+				<hardwareInterface>EffortJointInterface</hardwareInterface>
+			</joint>
+			<actuator name="${prefix}motor1">
+				<mechanicalReduction>1</mechanicalReduction>
+			</actuator>
+		</transmission>
+		<link name="${prefix}link1">
 			<collision>
 				<origin xyz="0 0 0" rpy="0 0 0"/>
@@ -50,5 +50,5 @@
 					<mesh filename="package://hdt_7dof_description/meshes/hdt_7dof_1_right.STL"/>
 				</geometry>
-				<material name="green"/>
+				<material name="${prefix}green"/>
 			</visual>
 			<inertial>
@@ -61,13 +61,13 @@
 			</inertial>
 		</link>
-		<gazebo reference="link1">
+		<gazebo reference="${prefix}link1">
 			<material>Gazebo/Green</material>
 		</gazebo>
-		<joint name="joint1f" type="fixed">
-			<parent link="link1"/>
-			<child link="link2a"/>
+		<joint name="${prefix}joint1f" type="fixed">
+			<parent link="${prefix}link1"/>
+			<child link="${prefix}link2a"/>
 			<origin xyz="-0.09217 0 0" rpy="0 0 0"/>
 		</joint>
-		<link name="link2a">
+		<link name="${prefix}link2a">
 			<collision>
 				<origin xyz="0 0 0" rpy="0 0 0"/>
@@ -81,5 +81,5 @@
 					<mesh filename="package://hdt_7dof_description/meshes/hdt_7dof_2a_right.STL"/>
 				</geometry>
-				<material name="black"/>
+				<material name="${prefix}black"/>
 			</visual>
 			<inertial>
@@ -92,27 +92,27 @@
 			</inertial>
 		</link>
-		<gazebo reference="link2a">
+		<gazebo reference="${prefix}link2a">
 			<material>Gazebo/Black</material>
 		</gazebo>
 		<!-- segment 2 -->
-		<joint name="joint2" type="revolute">
+		<joint name="${prefix}joint2" type="revolute">
 			<hdt id="42" kmin="100" kmax="200" inertia="0.1"/>
 			<axis xyz="0 1 0"/>
 			<limit effort="60.0" lower="-0.5236" upper="3.1416" velocity="2.0944"/>
 			<origin xyz="-0.07 0 0" rpy="0 0 0"/>
-			<parent link="link2a"/>
-			<child link="link2b"/>
-			<dynamics damping="0.7" friction="0.0"/>
-		</joint>
-		<transmission name="tran2">
-			<type>transmission_interface/SimpleTransmission</type>
-			<joint name="joint2">
-				<hardwareInterface>EffortJointInterface</hardwareInterface>
-			</joint>
-			<actuator name="motor2">
-				<mechanicalReduction>1</mechanicalReduction>
-			</actuator>
-		</transmission>
-		<link name="link2b">
+			<parent link="${prefix}link2a"/>
+			<child link="${prefix}link2b"/>
+			<dynamics damping="0.7" friction="0.0"/>
+		</joint>
+		<transmission name="${prefix}tran2">
+			<type>transmission_interface/SimpleTransmission</type>
+			<joint name="${prefix}joint2">
+				<hardwareInterface>EffortJointInterface</hardwareInterface>
+			</joint>
+			<actuator name="${prefix}motor2">
+				<mechanicalReduction>1</mechanicalReduction>
+			</actuator>
+		</transmission>
+		<link name="${prefix}link2b">
 			<collision>
 				<origin xyz="0 0 0" rpy="0 0 0"/>
@@ -126,5 +126,5 @@
 					<mesh filename="package://hdt_7dof_description/meshes/hdt_7dof_2b.STL"/>
 				</geometry>
-				<material name="grey"/>
+				<material name="${prefix}grey"/>
 			</visual>
 			<inertial>
@@ -137,27 +137,27 @@
 			</inertial>
 		</link>
-		<gazebo reference="link2b">
+		<gazebo reference="${prefix}link2b">
 			<material>Gazebo/Grey</material>
 		</gazebo>
 		<!-- segment 3 -->
-		<joint name="joint3" type="revolute">
+		<joint name="${prefix}joint3" type="revolute">
 			<hdt id="43" kmin="75" kmax="150" inertia="0.075"/>
 			<axis xyz="0 0 1"/>
 			<limit effort="60.0" lower="-2.0944" upper="2.0944" velocity="2.0944"/>
 			<origin xyz="0 0 -0.077" rpy="0 0 0" />
-			<parent link="link2b"/>
-			<child link="link3"/>
-			<dynamics damping="0.7" friction="0.0"/>
-		</joint>
-		<transmission name="tran3">
-			<type>transmission_interface/SimpleTransmission</type>
-			<joint name="joint3">
-				<hardwareInterface>EffortJointInterface</hardwareInterface>
-			</joint>
-			<actuator name="motor3">
-				<mechanicalReduction>1</mechanicalReduction>
-			</actuator>
-		</transmission>
-		<link name="link3">
+			<parent link="${prefix}link2b"/>
+			<child link="${prefix}link3"/>
+			<dynamics damping="0.7" friction="0.0"/>
+		</joint>
+		<transmission name="${prefix}tran3">
+			<type>transmission_interface/SimpleTransmission</type>
+			<joint name="${prefix}joint3">
+				<hardwareInterface>EffortJointInterface</hardwareInterface>
+			</joint>
+			<actuator name="${prefix}motor3">
+				<mechanicalReduction>1</mechanicalReduction>
+			</actuator>
+		</transmission>
+		<link name="${prefix}link3">
 			<collision>
 				<origin xyz="0 0 0.0" rpy="0 0 0"/>
@@ -171,5 +171,5 @@
 					<mesh filename="package://hdt_7dof_description/meshes/hdt_7dof_3.STL"/>
 				</geometry>
-				<material name="green"/>
+				<material name="${prefix}green"/>
 			</visual>
 			<inertial>
@@ -182,13 +182,13 @@
 			</inertial>
 		</link>
-		<gazebo reference="link3">
+		<gazebo reference="${prefix}link3">
 			<material>Gazebo/Green</material>
 		</gazebo>
-		<joint name="joint3f" type="fixed">
+		<joint name="${prefix}joint3f" type="fixed">
 			<origin xyz="0 0 -0.16271" rpy="0 0 0"/>
-			<parent link="link3"/>
-			<child link="link4a"/>
-		</joint>
-		<link name="link4a">
+			<parent link="${prefix}link3"/>
+			<child link="${prefix}link4a"/>
+		</joint>
+		<link name="${prefix}link4a">
 			<collision>
 				<origin xyz="0 0 0" rpy="0 0 0"/>
@@ -202,5 +202,5 @@
 					<mesh filename="package://hdt_7dof_description/meshes/hdt_7dof_4a.STL"/>
 				</geometry>
-				<material name="black"/>
+				<material name="${prefix}black"/>
 			</visual>
 			<inertial>
@@ -213,27 +213,27 @@
 			</inertial>
 		</link>
-		<gazebo reference="link4a">
+		<gazebo reference="${prefix}link4a">
 			<material>Gazebo/Black</material>
 		</gazebo>
 		<!-- segment 4 -->
-		<joint name="joint4" type="revolute">
+		<joint name="${prefix}joint4" type="revolute">
 			<hdt id="44" kmin="75" kmax="150" inertia="0.075"/>
 			<axis xyz="-1 0 0"/>
 			<limit effort="60.0" lower="-0.5236" upper="3.6652" velocity="2.0944"/>
 			<origin xyz="0 0 -0.07" rpy="3.1416 0 0"/>
-			<parent link="link4a"/>
-			<child link="link4b"/>
-			<dynamics damping="0.7" friction="0.0"/>
-		</joint>
-		<transmission name="tran4">
-			<type>transmission_interface/SimpleTransmission</type>
-			<joint name="joint4">
-				<hardwareInterface>EffortJointInterface</hardwareInterface>
-			</joint>
-			<actuator name="motor4">
-				<mechanicalReduction>1</mechanicalReduction>
-			</actuator>
-		</transmission>
-		<link name="link4b">
+			<parent link="${prefix}link4a"/>
+			<child link="${prefix}link4b"/>
+			<dynamics damping="0.7" friction="0.0"/>
+		</joint>
+		<transmission name="${prefix}tran4">
+			<type>transmission_interface/SimpleTransmission</type>
+			<joint name="${prefix}joint4">
+				<hardwareInterface>EffortJointInterface</hardwareInterface>
+			</joint>
+			<actuator name="${prefix}motor4">
+				<mechanicalReduction>1</mechanicalReduction>
+			</actuator>
+		</transmission>
+		<link name="${prefix}link4b">
 			<collision>
 				<origin xyz="0 0 0" rpy="0 0 0"/>
@@ -247,5 +247,5 @@
 					<mesh filename="package://hdt_7dof_description/meshes/hdt_7dof_4b.STL"/>
 				</geometry>
-				<material name="grey"/>
+				<material name="${prefix}grey"/>
 			</visual>
 			<inertial>
@@ -258,20 +258,20 @@
 			</inertial>
 		</link>
-		<gazebo reference="link4b">
+		<gazebo reference="${prefix}link4b">
 			<material>Gazebo/Grey</material>
 		</gazebo>
 		<!-- segment 5 -->
-		<joint name="joint5" type="revolute">
+		<joint name="${prefix}joint5" type="revolute">
 			<hdt id="45" kmin="50" kmax="100" inertia="0.05"/>
 			<axis xyz="0 -1 0"/>
 			<limit effort="60.0" lower="-2.0944" upper="2.0944" velocity="2.0944"/>
 			<origin xyz="0 -0.077 0" rpy="0 3.1416 0"/>
-			<parent link="link4b"/>
-			<child link="link5"/>
-			<dynamics damping="0.7" friction="0.0"/>
-		</joint>
-		<transmission name="tran5">
-			<type>transmission_interface/SimpleTransmission</type>
-			<joint name="joint5">
+			<parent link="${prefix}link4b"/>
+			<child link="${prefix}link5"/>
+			<dynamics damping="0.7" friction="0.0"/>
+		</joint>
+		<transmission name="${prefix}tran5">
+			<type>transmission_interface/SimpleTransmission</type>
+			<joint name="${prefix}joint5">
 				<hardwareInterface>EffortJointInterface</hardwareInterface>
 			</joint>
@@ -280,5 +280,5 @@
 			</actuator>
 		</transmission>
-		<link name="link5">
+		<link name="${prefix}link5">
 			<collision>
 				<origin xyz="0 0 0.0" rpy="0 0 0"/>
@@ -292,5 +292,5 @@
 					<mesh filename="package://hdt_7dof_description/meshes/hdt_7dof_5.STL"/>
 				</geometry>
-				<material name="green"/>
+				<material name="${prefix}green"/>
 			</visual>
 			<inertial>
@@ -303,13 +303,13 @@
 			</inertial>
 		</link>
-		<gazebo reference="link5">
+		<gazebo reference="${prefix}link5">
 			<material>Gazebo/Green</material>
 		</gazebo>
-		<joint name="joint5f" type="fixed">
+		<joint name="${prefix}joint5f" type="fixed">
 			<origin xyz="0 -0.09217 0" rpy="0 0 0"/>
-			<parent link="link5"/>
-			<child link="link6a"/>
-		</joint>
-		<link name="link6a">
+			<parent link="${prefix}link5"/>
+			<child link="${prefix}link6a"/>
+		</joint>
+		<link name="${prefix}link6a">
 			<collision>
 				<origin xyz="0 0 0" rpy="0 0 0"/>
@@ -323,5 +323,5 @@
 					<mesh filename="package://hdt_7dof_description/meshes/hdt_7dof_6a.STL"/>
 				</geometry>
-				<material name="black"/>
+				<material name="${prefix}black"/>
 			</visual>
 			<inertial>
@@ -334,27 +334,27 @@
 			</inertial>
 		</link>
-		<gazebo reference="link6a">
+		<gazebo reference="${prefix}link6a">
 			<material>Gazebo/Black</material>
 		</gazebo>
 		<!-- segment 6 -->
-		<joint name="joint6" type="revolute">
+		<joint name="${prefix}joint6" type="revolute">
 			<hdt id="46" kmin="50" kmax="100" inertia="0.05"/>
 			<axis xyz="1 0 0"/>
 			<limit effort="60.0" lower="-1.5708" upper="1.5708" velocity="2.0944"/>
 			<origin xyz="0 -0.055 0" rpy="0 0 0"/>
-			<parent link="link6a"/>
-			<child link="link6b"/>
-			<dynamics damping="0.7" friction="0.0"/>
-		</joint>
-		<transmission name="tran6">
-			<type>transmission_interface/SimpleTransmission</type>
-			<joint name="joint6">
-				<hardwareInterface>EffortJointInterface</hardwareInterface>
-			</joint>
-			<actuator name="motor6">
-				<mechanicalReduction>1</mechanicalReduction>
-			</actuator>
-		</transmission>
-		<link name="link6b">
+			<parent link="${prefix}link6a"/>
+			<child link="${prefix}link6b"/>
+			<dynamics damping="0.7" friction="0.0"/>
+		</joint>
+		<transmission name="${prefix}tran6">
+			<type>transmission_interface/SimpleTransmission</type>
+			<joint name="${prefix}joint6">
+				<hardwareInterface>EffortJointInterface</hardwareInterface>
+			</joint>
+			<actuator name="${prefix}motor6">
+				<mechanicalReduction>1</mechanicalReduction>
+			</actuator>
+		</transmission>
+		<link name="${prefix}link6b">
 			<collision>
 				<origin xyz="0 0 0" rpy="0 0 0"/>
@@ -368,5 +368,5 @@
 					<mesh filename="package://hdt_7dof_description/meshes/hdt_7dof_6b.STL"/>
 				</geometry>
-				<material name="grey"/>
+				<material name="${prefix}grey"/>
 			</visual>
 			<inertial>
@@ -379,27 +379,27 @@
 			</inertial>
 		</link>
-		<gazebo reference="link6b">
+		<gazebo reference="${prefix}link6b">
 			<material>Gazebo/Grey</material>
 		</gazebo>
 		<!-- segment 7 -->
-		<joint name="joint7" type="revolute">
+		<joint name="${prefix}joint7" type="revolute">
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
File: urdf/hdt_7dof_right.xacro (robot description, xacro)
@@ -9,4 +9,4 @@
 	<link name="world" />
 	<xacro:include filename="$(find hdt_7dof_description)/urdf/hdt_7dof_right_macro.xacro" />
-	<xacro:hdt_7dof_right parent="world" x="0" y="0" z="0" />
+	<xacro:hdt_7dof_right parent="world" x="0" y="0" z="0" yaw="1.57079" prefix="" />
 </robot>
