Commit message: give left and right macros a default yaw

File: urdf/hdt_7dof_left.xacro (robot description, xacro)
@@ -9,4 +9,4 @@
 	<link name="world" />
 	<xacro:include filename="$(find hdt_7dof_description)/urdf/hdt_7dof_macro.xacro" />
-	<xacro:hdt_7dof_left parent="world" x="0" y="0" z="0" yaw="-1.57079" prefix="l_" motor_base_id="51" />
+	<xacro:hdt_7dof_left parent="world" x="0" y="0" z="0" prefix="l_" motor_base_id="51" />
 </robot>

File: urdf/hdt_7dof_macro.xacro (robot description, xacro)
@@ -1,9 +1,9 @@
 <?xml version="1.0"?>
 <robot name="hdt_7dof" xmlns:xacro="http://www.ros.org/wiki/xacro">
-	<xacro:macro name="hdt_7dof_left" params="prefix parent x y z yaw motor_base_id">
-		<xacro:hdt_7dof reflect="1" left_only="1" right_only="0" prefix="${prefix}" parent="${parent}" x="${x}" y="${y}" z="${z}" yaw="${yaw}" motor_base_id="${motor_base_id}"/>
+	<xacro:macro name="hdt_7dof_left" params="prefix parent x y z motor_base_id">
+		<xacro:hdt_7dof reflect="1" left_only="1" right_only="0" prefix="${prefix}" parent="${parent}" x="${x}" y="${y}" z="${z}" yaw="-1.57079" motor_base_id="${motor_base_id}"/>
 	</xacro:macro>
-	<xacro:macro name="hdt_7dof_right" params="prefix parent x y z yaw motor_base_id">
-		<xacro:hdt_7dof reflect="-1" left_only="0" right_only="1" prefix="${prefix}" parent="${parent}" x="${x}" y="${y}" z="${z}" yaw="${yaw}" motor_base_id="${motor_base_id}"/>
+	<xacro:macro name="hdt_7dof_right" params="prefix parent x y z motor_base_id">
+		<xacro:hdt_7dof reflect="-1" left_only="0" right_only="1" prefix="${prefix}" parent="${parent}" x="${x}" y="${y}" z="${z}" yaw="1.57079" motor_base_id="${motor_base_id}"/>
 	</xacro:macro>
 	<!-- default inertia -->

File: urdf/hdt_7dof_right.xacro (robot description, xacro)
@@ -9,4 +9,4 @@
 	<link name="world" />
 	<xacro:include filename="$(find hdt_7dof_description)/urdf/hdt_7dof_macro.xacro" />
-	<xacro:hdt_7dof_right parent="world" x="0" y="0" z="0" yaw="1.57079" prefix="r_" motor_base_id="1" />
+	<xacro:hdt_7dof_right parent="world" x="0" y="0" z="0" prefix="r_" motor_base_id="1" />
 </robot>

Commit message: added endpoint link to urdf

File: urdf/hdt_7dof_left.xacro (robot description, xacro)
@@ -423,4 +423,12 @@
 		<material>Gazebo/Black</material>
 	</gazebo>
+	<!-- endpoint -->
+	<joint name="endpoint_joint" type="fixed">
+		<origin xyz="0 -0.055 0" rpy="0 0 0"/>
+		<parent link="link7"/>
+		<child link="endpoint_link"/>
+	</joint>
+	<link name="endpoint_link">
+	</link>
 	<!-- palm -->
 	<joint name="palm" type="fixed">
